File: 04-line/04-line.kicad_sch (KiCad schematic)
At the start: 71 parts, among them J1 Conn_01x10, J2 Conn_01x10, J3 Conn_01x08

Commit message: 全国行きたかった
Parts:
- removed U1, U10, U11, U12, U13, U14, U15, U16, U17, U18, U19, U2, U20, U21, U22, U3, U4, U5, U6, U7, U8, U9: ~, Akiduki:RPR220, symbol akiduki:RPR220
- added U1, U10, U11, U12, U13, U14, U15, U16, U17, U18, U19, U2, U20, U21, U25, U3, U4, U5, U6, U7, U8, U9: ~, symbol akiduki:LBR127HLD
- R1, R10, R11, R12, R17, R19, R20, R21, R22, R23, R24, R25, R26, R27, R3, R37, R38, R39, R40, R5, R6, R9: value 30 -> 105
Connections:
- net +3V3: now also U1.1 (Anode), U10.1 (Anode), U11.1 (Anode), U12.1 (Anode), U13.1 (Anode), U14.1 (Anode), U15.1 (Anode), U16.1 (Anode), U17.1 (Anode), U18.1 (Anode), U19.1 (Anode), U2.1 (Anode), U20.1 (Anode), U21.1 (Anode), U25.1 (Anode), U3.1 (Anode), U4.1 (Anode), U5.1 (Anode), U6.1 (Anode), U7.1 (Anode), U8.1 (Anode), U9.1 (Anode)
- net GND: now also U1.3 (Emitter), U10.3 (Emitter), U11.3 (Emitter), U12.3 (Emitter), U13.3 (Emitter), U14.3 (Emitter), U15.3 (Emitter), U16.3 (Emitter), U17.3 (Emitter), U18.3 (Emitter), U19.3 (Emitter), U2.3 (Emitter), U20.3 (Emitter), U21.3 (Emitter), U25.3 (Emitter), U3.3 (Emitter), U4.3 (Emitter), U5.3 (Emitter), U6.3 (Emitter), U7.3 (Emitter), U8.3 (Emitter), U9.3 (Emitter)
- net photo_LL: now also U20.4 (Collector)
- net photo_L_1: now also U25.4 (Collector)
- net photo_L_2: now also U1.4 (Collector)
- net photo_L_3: now also U2.4 (Collector)
- net photo_L_4: now also U3.4 (Collector)
- net photo_L_5: now also U4.4 (Collector)
- net photo_L_6: now also U5.4 (Collector)
- net photo_L_7: now also U6.4 (Collector)
- net photo_L_8: now also U7.4 (Collector)
- net photo_L_9: now also U8.4 (Collector)
- net photo_RR: now also U21.4 (Collector)
- net photo_R_1: now also U9.4 (Collector)
- net photo_R_2: now also U10.4 (Collector)
- net photo_R_3: now also U11.4 (Collector)
- net photo_R_4: now also U12.4 (Collector)
- net photo_R_5: now also U13.4 (Collector)
- net photo_R_6: now also U14.4 (Collector)
- net photo_R_7: now also U15.4 (Collector)
- net photo_R_8: now also U16.4 (Collector)
- net photo_R_9: now also U17.4 (Collector)
- net photo_center: now also U18.4 (Collector)
- net photo_front: now also U19.4 (Collector)
- net at R11.1: now also U6.2 (Cathode)
- net at R22.1: now also U12.2 (Cathode)
- net at R3.1: now also U1.2 (Cathode)
- net at R23.1: now also U13.2 (Cathode)
- net at R20.1: now also U10.2 (Cathode)
- net at R19.1: now also U9.2 (Cathode)
- net at R26.1: now also U16.2 (Cathode)
- net at R5.1: now also U2.2 (Cathode)
- net at R10.1: now also U5.2 (Cathode)
- net at R38.1: now also U19.2 (Cathode)
- net at R27.1: now also U17.2 (Cathode)
- net at R37.1: now also U18.2 (Cathode)
- net at R1.1: now also U25.2 (Cathode)
- net at R21.1: now also U11.2 (Cathode)
- net at R24.1: now also U14.2 (Cathode)
- net at R17.1: now also U8.2 (Cathode)
- net at R39.1: now also U20.2 (Cathode)
- net at R9.1: now also U4.2 (Cathode)
- net at R25.1: now also U15.2 (Cathode)
- net at R12.1: now also U7.2 (Cathode)
- net at R40.1: now also U21.2 (Cathode)
- net at R6.1: now also U3.2 (Cathode)

Commit message: がんばる
Parts:
- removed J1, J2: Conn_01x10, Connector_PinHeader_2.54mm:PinHeader_1x10_P2.54mm_Vertical, symbol Connector_Generic:Conn_01x10
- removed J3: Conn_01x08, Connector_PinHeader_2.54mm:PinHeader_1x08_P2.54mm_Vertical, symbol Connector_Generic:Conn_01x08
- removed R12, R17, R26, R27: 105, symbol Device:R
- removed R16, R18, R35, R36: 1k, symbol Device:R
- removed U16, U17, U7, U8: ~, symbol akiduki:LBR127HLD
- removed U23, U24: ~, S11059:S11059, symbol S11059:S11059
- added C1: 100n, symbol Device:C
- added C10: 100u, symbol Device:C
- added C2: 4.7u, symbol Device:C
- added C3, C6: 0.1u, symbol Device:C
- added C4, C5: 1u, symbol Device:C
- added C7, C8: 10u, symbol Device:C
- added C9: 0.33u, symbol Device:C
- added D1, D2, D3, D4: WS2812B, LED_SMD:LED_WS2812B_PLCC4_5.0x5.0mm_P3.2mm, symbol LED:WS2812B
- added J2: VL53L0X, Connector_PinHeader_2.54mm:PinHeader_1x04_P2.54mm_Vertical, symbol Connector_Generic:Conn_01x04
- added J2: WRITER CONN, Connector_PinHeader_2.54mm:PinHeader_2x04_P2.54mm_Vertical, symbol Connector_Generic:Conn_02x04_Counter_Clockwise
- added J3: ToMAIN, Connector_JST:JST_XH_B4B-XH-A_1x04_P2.50mm_Vertical, symbol Connector_Generic:Conn_01x04
- added R38, R39: 100k, symbol Device:R
- added R5: 10k, Resistor_SMD:R_0805_2012Metric, symbol Device:R
- added U1, U11, U21, U22, U23: ~, Package_SO:SOIC-14_3.9x8.7mm_P1.27mm, symbol JLCPCB_items:LM2901DR
- added U24: STM32F446RETx, Package_QFP:LQFP-64_10x10mm_P0.5mm, symbol MCU_ST_STM32F4:STM32F446RETx
- added U25, U26: ~, Akiduki:S11059, symbol akiduki:S11059
- added U27: ~, Package_TO_SOT_SMD:SOT-223-6, symbol JLCPCB_items:TPS7A4533DCQR
- added U28: ~, Package_TO_SOT_SMD:TO-252-3_TabPin2, symbol JLCPCB_items:BA50BC0FP
- R1, R19, R20, R21, R22, R23, R24, R25: footprint (none) -> Resistor_SMD:R_0603_1608Metric; LCSC (none) -> C128061
- R10: renamed from R2; footprint (none) -> Resistor_SMD:R_1206_3216Metric; LCSC (none) -> C138242
- R11: renamed from R4; footprint (none) -> Resistor_SMD:R_1206_3216Metric; LCSC (none) -> C138242
- R12: renamed from R7; footprint (none) -> Resistor_SMD:R_1206_3216Metric; LCSC (none) -> C138242
- R13: renamed from R8; footprint (none) -> Resistor_SMD:R_1206_3216Metric; LCSC (none) -> C138242
- R14: renamed from R13; footprint (none) -> Resistor_SMD:R_1206_3216Metric; LCSC (none) -> C138242
- R15: renamed from R14; footprint (none) -> Resistor_SMD:R_1206_3216Metric; LCSC (none) -> C138242
- R16: renamed from R15; footprint (none) -> Resistor_SMD:R_1206_3216Metric; LCSC (none) -> C138242
- R17: renamed from R41; footprint (none) -> Resistor_SMD:R_1206_3216Metric; LCSC (none) -> C138242
- R18: renamed from R42; footprint (none) -> Resistor_SMD:R_1206_3216Metric; LCSC (none) -> C138242
- R2: renamed from R3; footprint (none) -> Resistor_SMD:R_0603_1608Metric; LCSC (none) -> C128061
- R26: renamed from R39; footprint (none) -> Resistor_SMD:R_0603_1608Metric; LCSC (none) -> C128061
- R27: renamed from R40; footprint (none) -> Resistor_SMD:R_0603_1608Metric; LCSC (none) -> C128061
- R28, R29, R30, R31, R32, R33, R34: footprint (none) -> Resistor_SMD:R_1206_3216Metric; LCSC (none) -> C138242
- R3: renamed from R5; footprint (none) -> Resistor_SMD:R_0603_1608Metric; LCSC (none) -> C128061
- R35: renamed from R43; footprint (none) -> Resistor_SMD:R_1206_3216Metric; LCSC (none) -> C138242
- R36: renamed from R44; footprint (none) -> Resistor_SMD:R_1206_3216Metric; LCSC (none) -> C138242
- R4: renamed from R6; footprint (none) -> Resistor_SMD:R_0603_1608Metric; LCSC (none) -> C128061
- R5: renamed from R9; footprint (none) -> Resistor_SMD:R_0603_1608Metric; LCSC (none) -> C128061
- R6: renamed from R10; footprint (none) -> Resistor_SMD:R_0603_1608Metric; LCSC (none) -> C128061
- R7: renamed from R11; footprint (none) -> Resistor_SMD:R_0603_1608Metric; LCSC (none) -> C128061
- R8: renamed from R37; footprint (none) -> Resistor_SMD:R_0603_1608Metric; LCSC (none) -> C128061
- R9: renamed from R38; footprint (none) -> Resistor_SMD:R_0603_1608Metric; LCSC (none) -> C128061
- U10: renamed from U19; footprint (none) -> Akiduki:LBR127HLD
- U12: renamed from U9; footprint (none) -> Akiduki:LBR127HLD
- U13: renamed from U10; footprint (none) -> Akiduki:LBR127HLD
- U14: renamed from U11; footprint (none) -> Akiduki:LBR127HLD
- U15: renamed from U12; footprint (none) -> Akiduki:LBR127HLD
- U16: renamed from U13; footprint (none) -> Akiduki:LBR127HLD
- U17: renamed from U14; footprint (none) -> Akiduki:LBR127HLD
- U18: renamed from U15; footprint (none) -> Akiduki:LBR127HLD
- U19: renamed from U20; footprint (none) -> Akiduki:LBR127HLD
- U2: renamed from U25; footprint (none) -> Akiduki:LBR127HLD
- U20: renamed from U21; footprint (none) -> Akiduki:LBR127HLD
- U3: renamed from U1; footprint (none) -> Akiduki:LBR127HLD
- U4: renamed from U2; footprint (none) -> Akiduki:LBR127HLD
- U5: renamed from U3; footprint (none) -> Akiduki:LBR127HLD
- U6: renamed from U4; footprint (none) -> Akiduki:LBR127HLD
- U7: renamed from U5; footprint (none) -> Akiduki:LBR127HLD
- U8: renamed from U6; footprint (none) -> Akiduki:LBR127HLD
- U9: renamed from U18; footprint (none) -> Akiduki:LBR127HLD
Connections:
- net +3V3: now also C3.1, C6.1, C8.1, J2.1 (Pin_1), J2.8 (Pin_8), U1.3 (VCC), U11.3 (VCC), U21.3 (VCC), U22.3 (VCC), U23.3 (VCC), U24.1 (VBAT), U24.13 (VDDA), U24.19 (VDD), U24.32 (VDD), U24.48 (VDD), U24.64 (VDD), U25.1 (VDD), U26.1 (VDD), U27.4 (OUT), U27.5 (SENSE)
- net GND: now also C1.1, C10.2, C2.2, C3.2, C4.2, C5.2, C6.2, C7.2, C8.2, C9.2, D1.3 (VSS), D2.3 (VSS), D3.3 (VSS), D4.3 (VSS), J2.2 (Pin_2), J2.6 (Pin_6), J3.2 (Pin_2), R5.2, U1.12 (GND), U11.12 (GND), U21.12 (GND), U22.12 (GND), U23.12 (GND), U24.12 (VSSA), U24.18 (VSS), U24.31 (VSS), U24.47 (VSS), U24.63 (VSS), U25.5 (GND), U26.5 (GND), U27.3 (GND), U27.6 (GND), U28.2 (GND)
- net I2C1_SCL: now also J2.3 (Pin_3), U24.58 (PB6), U26.6 (SCL)
- net I2C1_SDA: now also J2.4 (Pin_4), U24.59 (PB7), U26.10 (SDA)
- net I2C2_SCL: now also U24.29 (PB10), U25.6 (SCL)
- net I2C2_SDA: now also U24.53 (PC12), U25.10 (SDA)
- net photo_LL: now also U22.7 (1IN+)
- net photo_L_1: now also U1.7 (1IN+)
- net photo_L_2: now also U1.5 (2IN+)
- net photo_L_3: now also U1.9 (3IN+)
- net photo_L_4: now also U1.11 (4IN+)
- net photo_L_5: now also U11.7 (1IN+)
- net photo_L_6: now also U11.5 (2IN+)
- net photo_L_7: now also U11.9 (3IN+)
- net photo_RR: now also U22.5 (2IN+)
- net photo_R_1: now also U21.7 (1IN+)
- net photo_R_2: now also U21.5 (2IN+)
- net photo_R_3: now also U21.9 (3IN+)
- net photo_R_4: now also U21.11 (4IN+)
- net photo_R_5: now also U23.7 (1IN+)
- net photo_R_6: now also U23.5 (2IN+)
- net photo_R_7: now also U23.9 (3IN+)
- net photo_center: now also U11.11 (4IN+)
- net photo_front: now also U23.11 (4IN+)
- new net: D2.2 (DOUT), D3.4 (DIN)
- new net: D1.2 (DOUT), D2.4 (DIN)
- new net: D1.4 (DIN), U24.33 (PB12)
- new net: R39.1, U24.41 (PA8)
- new net: R38.1, U24.22 (PA6)
- new net: C2.1, U24.30 (VCAP_1)
- new net: D3.2 (DOUT), D4.4 (DIN)
- new net +5V: C10.1, D1.1 (VDD), D2.1 (VDD), D3.1 (VDD), D4.1 (VDD), U28.3 (OUT)
- new net Ag_Com: C4.1, R38.2, U22.4 (2IN-), U22.6 (1IN-)
- new net BOOT0: J2.5 (Pin_5), R5.1, U24.60 (BOOT0)
- new net B_W_Com: C5.1, R39.2, U1.10 (4IN-), U1.4 (2IN-), U1.6 (1IN-), U1.8 (3IN-), U11.10 (4IN-), U11.4 (2IN-), U11.6 (1IN-), U11.8 (3IN-), U21.10 (4IN-), U21.4 (2IN-), U21.6 (1IN-), U21.8 (3IN-), U23.10 (4IN-), U23.4 (2IN-), U23.6 (1IN-), U23.8 (3IN-)
- new net LL_OUT: U22.1 (OUT1), U24.35 (PB14)
- new net L_1_OUT: U1.1 (OUT1), U24.57 (PB5)
- new net L_2_OUT: U1.2 (OUT2), U24.56 (PB4)
- new net L_3_OUT: U1.14 (OUT3), U24.55 (PB3)
- new net L_4_OUT: U1.13 (OUT4), U24.54 (PD2)
- new net L_5_OUT: U11.1 (OUT1), U24.52 (PC11)
- new net L_6_OUT: U11.2 (OUT2), U24.51 (PC10)
- new net L_7_OUT: U11.14 (OUT3), U24.50 (PA15)
- new net NRST: C1.2, J2.3 (Pin_3), U24.7 (NRST)
- new net RR_OUT: U22.2 (OUT2), U24.34 (PB13)
- new net R_1_OUT: U21.2 (OUT2), U24.36 (PB15)
- new net R_2_OUT: U21.1 (OUT1), U24.37 (PC6)
- new net R_3_OUT: U21.14 (OUT3), U24.38 (PC7)
- new net R_4_OUT: U21.13 (OUT4), U24.39 (PC8)
- new net R_5_OUT: U23.1 (OUT1), U24.40 (PC9)
- new net R_6_OUT: U23.2 (OUT2), U24.44 (PA11)
- new net R_7_OUT: U23.14 (OUT3), U24.45 (PA12)
- new net UART1_RX: J2.2 (Pin_2), U24.43 (PA10)
- new net UART1_TX: J2.4 (Pin_4), U24.42 (PA9)
- new net UART2_RX: J3.3 (Pin_3), U24.17 (PA3)
- new net UART2_TX: J3.4 (Pin_4), U24.16 (PA2)
- new net VDD: C7.1, C9.1, J3.1 (Pin_1), U27.1 (SHDN), U27.2 (IN), U28.1 (IN)
- new net center_OUT: U11.13 (OUT4), U24.49 (PA14)
- new net front_OUT: U23.13 (OUT4), U24.46 (PA13)
- no-connect marks 0 -> 30
Other:
- title: (none) -> 04-LINE
- moved on the sheet: R1, R10, R11, R12, R13, R14, R15, R16, R17, R18, R19, R2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

Commit message: line...
Parts:
- C1, C10, C2, C3, C4, C5, C6, C7, C8, C9: footprint (none) -> Capacitor_SMD:C_0805_2012Metric
- R38, R39: footprint (none) -> Resistor_SMD:R_0805_2012Metric
Changed lines of the file:
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@@
       (effects (font (size 1.27 1.27)) (justify left))
     )
-    (property "Footprint" "" (at 200.3552 154.305 0)
+    (property "Footprint" "Capacitor_SMD:C_0805_2012Metric" (at 200.3552 154.305 0)
       (effects (font (size 1.27 1.27)) hide)
     )
@@
       (effects (font (size 1.27 1.27)) (justify left))
     )
-    (property "Footprint" "" (at 229.5652 27.305 0)
+    (property "Footprint" "Capacitor_SMD:C_0805_2012Metric" (at 229.5652 27.305 0)
       (effects (font (size 1.27 1.27)) hide)
     )
@@
       (effects (font (size 1.27 1.27)) (justify left))
     )
-    (property "Footprint" "" (at 163.5252 42.545 0)
+    (property "Footprint" "Capacitor_SMD:C_0805_2012Metric" (at 163.5252 42.545 0)
       (effects (font (size 1.27 1.27)) hide)
     )
@@
       (effects (font (size 1.27 1.27)) (justify left))
     )
-    (property "Footprint" "" (at 192.1002 27.305 0)
+    (property "Footprint" "Capacitor_SMD:C_0805_2012Metric" (at 192.1002 27.305 0)
       (effects (font (size 1.27 1.27)) hide)
     )
@@
       (effects (font (size 1.27 1.27)) (justify left))
     )
-    (property "Footprint" "" (at 232.7402 54.61 0)
+    (property "Footprint" "Capacitor_SMD:C_0805_2012Metric" (at 232.7402 54.61 0)
       (effects (font (size 1.27 1.27)) hide)
     )
@@
       (effects (font (size 1.27 1.27)) (justify left))
     )
-    (property "Footprint" "" (at 273.3802 27.94 0)
+    (property "Footprint" "Capacitor_SMD:C_0805_2012Metric" (at 273.3802 27.94 0)
       (effects (font (size 1.27 1.27)) hide)
     )
@@
       (effects (font (size 1.27 1.27)) (justify left))
     )
-    (property "Footprint" "" (at 250.5202 27.94 0)
+    (property "Footprint" "Capacitor_SMD:C_0805_2012Metric" (at 250.5202 27.94 0)
       (effects (font (size 1.27 1.27)) hide)
     )
@@
       (effects (font (size 1.27 1.27)))
     )
-    (property "Footprint" "" (at 226.06 70.358 90)
+    (property "Footprint" "Resistor_SMD:R_0805_2012Metric" (at 226.06 70.358 90)
       (effects (font (size 1.27 1.27)) hide)
     )
@@
       (effects (font (size 1.27 1.27)))
     )
-    (property "Footprint" "" (at 226.06 48.768 90)
+    (property "Footprint" "Resistor_SMD:R_0805_2012Metric" (at 226.06 48.768 90)
       (effects (font (size 1.27 1.27)) hide)
     )
@@
       (effects (font (size 1.27 1.27)) (justify left))
     )
-    (property "Footprint" "" (at 232.7402 76.2 0)
+    (property "Footprint" "Capacitor_SMD:C_0805_2012Metric" (at 232.7402 76.2 0)
       (effects (font (size 1.27 1.27)) hide)
     )
@@
       (effects (font (size 1.27 1.27)) (justify left))
     )
-    (property "Footprint" "" (at 243.5352 154.305 0)
+    (property "Footprint" "Capacitor_SMD:C_0805_2012Metric" (at 243.5352 154.305 0)
       (effects (font (size 1.27 1.27)) hide)
     )
@@
       (effects (font (size 1.27 1.27)) (justify left))
     )
-    (property "Footprint" "" (at 164.1602 116.205 0)
+    (property "Footprint" "Capacitor_SMD:C_0805_2012Metric" (at 164.1602 116.205 0)
       (effects (font (size 1.27 1.27)) hide)
     )

Commit message: ラインセンサ完成
Parts:
- removed R27: 105, Resistor_SMD:R_0603_1608Metric, symbol Device:R
- removed R35, R36: 1k, Resistor_SMD:R_1206_3216Metric, symbol Device:R
- removed R38, R39: 100k, Resistor_SMD:R_0805_2012Metric, symbol Device:R
- removed U1, U11, U21, U22, U23: ~, Package_SO:SOIC-14_3.9x8.7mm_P1.27mm, symbol JLCPCB_items:LM2901DR
- removed U19, U20: ~, Akiduki:LBR127HLD, symbol akiduki:LBR127HLD
- added C11, C12, C13, C15: 100n, Capacitor_SMD:C_0402_1005Metric, symbol Device:C
- added C14: 4.7u, Capacitor_SMD:C_0402_1005Metric, symbol Device:C
- added C16: 1u, Capacitor_SMD:C_0402_1005Metric, symbol Device:C
- added D5, D6, D7, D8: WS2812B, LED_SMD:LED_WS2812B_PLCC4_5.0x5.0mm_P3.2mm, symbol LED:WS2812B
- added FB1: FerriteBead, Resistor_SMD:R_0805_2012Metric, symbol Device:FerriteBead
- added J1: ST-LINK, Connector_PinHeader_2.54mm:PinHeader_1x04_P2.54mm_Vertical, symbol Connector_Generic:Conn_01x04
- added J5: SSD1306, Connector_PinHeader_2.54mm:PinHeader_1x04_P2.54mm_Vertical, symbol Connector_Generic:Conn_01x04
- C1: footprint Capacitor_SMD:C_0805_2012Metric -> Capacitor_SMD:C_0402_1005Metric; LCSC (none) -> C1525
- C10: footprint Capacitor_SMD:C_0805_2012Metric -> Capacitor_SMD:C_1206_3216Metric; LCSC (none) -> C7432784
- C2: footprint Capacitor_SMD:C_0805_2012Metric -> Capacitor_SMD:C_0402_1005Metric; LCSC (none) -> C23733
- C3, C6: value 0.1u -> 100n; footprint Capacitor_SMD:C_0805_2012Metric -> Capacitor_SMD:C_0402_1005Metric; LCSC (none) -> C1525
- C4, C5: value 1u -> 100n; footprint Capacitor_SMD:C_0805_2012Metric -> Capacitor_SMD:C_0402_1005Metric; LCSC (none) -> C1525
- C7, C8: footprint Capacitor_SMD:C_0805_2012Metric -> Capacitor_SMD:C_0603_1608Metric; LCSC (none) -> C19702
- C9: LCSC (none) -> C2961026
- D1, D2, D3, D4: LCSC (none) -> C2843785
- R26: value 105 -> 10k; LCSC C128061 -> C137819
- R5: footprint Resistor_SMD:R_0805_2012Metric -> Resistor_SMD:R_0603_1608Metric; LCSC C17414 -> C137819
- U24: LCSC (none) -> C69336
- U27: LCSC (none) -> C2877942
- U28: LCSC (none) -> C2909275
Connections:
- net Ag_Com is gone; now on net GND: C4.1
- net B_W_Com is gone; now on net GND: C5.1
- net +3V3: now also C4.2, C5.2, C11.2, C12.2, C13.2, C14.1, FB1.1, J5.2 (Pin_2); no longer U24.13 (VDDA)
- net +5V: now also D5.1 (VDD), D6.1 (VDD), D7.1 (VDD), D8.1 (VDD)
- net GND: now also C11.1, C12.1, C13.1, C14.2, C15.1, C16.1, D5.3 (VSS), D6.3 (VSS), D7.3 (VSS), D8.3 (VSS), J1.4 (Pin_4), J5.1 (Pin_1); no longer C4.2, C5.2
- net I2C1_SCL: no longer J2.3 (Pin_3)
- net I2C1_SDA: no longer J2.4 (Pin_4)
- net NRST: now also J1.3 (Pin_3)
- net photo_L_1: now also U24.16 (PA2)
- net photo_L_2: now also U24.15 (PA1)
- net photo_L_3: now also U24.14 (PA0)
- net photo_L_4: now also U24.11 (PC3)
- net photo_L_5: now also U24.10 (PC2)
- net photo_L_6: now also U24.9 (PC1)
- net photo_L_7: now also U24.8 (PC0)
- net photo_R_1: now also U24.21 (PA5)
- net photo_R_2: now also U24.22 (PA6)
- net photo_R_3: now also U24.23 (PA7)
- net photo_R_4: now also U24.24 (PC4)
- net photo_R_5: now also U24.25 (PC5)
- net photo_R_6: now also U24.26 (PB0)
- net photo_R_7: now also U24.27 (PB1)
- net photo_center: now also U24.20 (PA4)
- net photo_front: now also U24.17 (PA3)
- net at R26.1: now also U24.28 (PB2)
- net at U24.33 (PB12): no longer D1.4 (DIN)
- net I2C3_SCL: now reaches U24.41 (PA8)
- net I2C3_SCL: now also J2.3 (Pin_3), J5.3 (Pin_3)
- net LED_R: now reaches U24.3 (PC14)
- net LED_R: now also D5.4 (DIN)
- net LED_L: now reaches U24.4 (PC15)
- net LED_L: now also D1.4 (DIN)
- net LL_OUT: no longer names the net of U24.35 (PB14)
- net L_1_OUT: no longer names the net of U24.57 (PB5)
- net L_2_OUT: no longer names the net of U24.56 (PB4)
- net L_3_OUT: no longer names the net of U24.55 (PB3)
- net L_4_OUT: no longer names the net of U24.54 (PD2)
- net L_5_OUT renamed UART3_RX
- net UART3_RX: now also J3.3 (Pin_3)
- net L_6_OUT renamed UART3_TX
- net UART3_TX: now also J3.4 (Pin_4)
- net L_7_OUT: no longer names the net of U24.50 (PA15)
- net RR_OUT: no longer names the net of U24.34 (PB13)
- net R_1_OUT: no longer names the net of U24.36 (PB15)
- net R_2_OUT: no longer names the net of U24.37 (PC6)
- net R_3_OUT: no longer names the net of U24.38 (PC7)
- net R_4_OUT: no longer names the net of U24.39 (PC8)
- net R_5_OUT renamed I2C3_SDA
- net I2C3_SDA: now also J2.4 (Pin_4), J5.4 (Pin_4)
- net R_6_OUT: no longer names the net of U24.44 (PA11)
- net R_7_OUT: no longer names the net of U24.45 (PA12)
- removed net UART2_RX: J3.3 (Pin_3), U24.17 (PA3)
- removed net UART2_TX: J3.4 (Pin_4), U24.16 (PA2)
- net center_OUT renamed SWCLK
- net SWCLK: now also J1.1 (Pin_1)
- net front_OUT renamed SWDIO
- net SWDIO: now also J1.2 (Pin_2)
- new net: C15.2, C16.2, FB1.2, U24.13 (VDDA)
- new net: D5.2 (DOUT), D6.4 (DIN)
- new net: D6.2 (DOUT), D7.4 (DIN)
- new net: D7.2 (DOUT), D8.4 (DIN)
- no-connect marks 30 -> 23
Other:
- company: (none) -> tuton
- moved on the sheet: C1, C10, C2, C3, C6, C7, C8, C9, D1, D2, D3, D4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

Commit message: 前けずった
Parts:
- removed D3, D7: WS2812B, LED_SMD:LED_WS2812B_PLCC4_5.0x5.0mm_P3.2mm, symbol LED:WS2812B
- removed J2: VL53L0X, Connector_PinHeader_2.54mm:PinHeader_1x04_P2.54mm_Vertical, symbol Connector_Generic:Conn_01x04
- removed J5: SSD1306, Connector_PinHeader_2.54mm:PinHeader_1x04_P2.54mm_Vertical, symbol Connector_Generic:Conn_01x04
Connections:
- net at D2.2 (DOUT): now also D4.4 (DIN)
- net at D6.2 (DOUT): now also D8.4 (DIN)
Other:
- moved on the sheet: D4, D8

Commit message: いっぱい増えた
Parts:
- removed C1, C11, C12, C13, C15, C4, C5: 100n, Capacitor_SMD:C_0402_1005Metric, symbol Device:C
- removed C10: 100u, Capacitor_SMD:C_1206_3216Metric, symbol Device:C
- removed C14, C2: 4.7u, Capacitor_SMD:C_0402_1005Metric, symbol Device:C
- removed C16: 1u, Capacitor_SMD:C_0402_1005Metric, symbol Device:C
- removed C7, C8: 10u, Capacitor_SMD:C_0603_1608Metric, symbol Device:C
- removed C9: 0.33u, Capacitor_SMD:C_0805_2012Metric, symbol Device:C
- removed FB1: FerriteBead, Resistor_SMD:R_0805_2012Metric, symbol Device:FerriteBead
- removed J1: ST-LINK, Connector_PinHeader_2.54mm:PinHeader_1x04_P2.54mm_Vertical, symbol Connector_Generic:Conn_01x04
- removed J2: WRITER CONN, Connector_PinHeader_2.54mm:PinHeader_2x04_P2.54mm_Vertical, symbol Connector_Generic:Conn_02x04_Counter_Clockwise
- removed J3: ToMAIN, Connector_JST:JST_XH_B4B-XH-A_1x04_P2.50mm_Vertical, symbol Connector_Generic:Conn_01x04
- removed R26, R5: 10k, Resistor_SMD:R_0603_1608Metric, symbol Device:R
- removed U24: STM32F446RETx, Package_QFP:LQFP-64_10x10mm_P0.5mm, symbol MCU_ST_STM32F4:STM32F446RETx
- removed U27: ~, Package_TO_SOT_SMD:SOT-223-6, symbol JLCPCB_items:TPS7A4533DCQR
- removed U28: ~, Package_TO_SOT_SMD:TO-252-3_TabPin2, symbol JLCPCB_items:BA50BC0FP
- added J1: Conn_01x18, Connector_PinHeader_2.54mm:PinHeader_1x18_P2.54mm_Vertical, symbol Connector_Generic:Conn_01x18
- added J3: CS_R, Connector_PinHeader_2.54mm:PinHeader_2x03_P2.54mm_Vertical, symbol Connector_Generic:Conn_02x03_Counter_Clockwise
- added J5: CS_L, Connector_PinHeader_2.54mm:PinHeader_2x03_P2.54mm_Vertical, symbol Connector_Generic:Conn_02x03_Counter_Clockwise
- R1, R19, R2, R20, R21, R22, R23, R24, R25, R3, R4, R5, R6, R7, R8, R9: value 105 -> 120; LCSC C128061 -> C22787
- R10, R11, R12, R13, R14, R15, R16, R17, R18, R28, R29, R30, R31, R32, R33, R34: footprint Resistor_SMD:R_1206_3216Metric -> Resistor_SMD:R_0603_1608Metric; LCSC C138242 -> C21190
Connections:
- net +3V3: now also J1.18 (Pin_18); no longer C3.1, C6.1, U25.1 (VDD), U26.1 (VDD)
- net GND: now also U25.2 (GND), U25.3 (GND), U25.4 (GND), U25.7 (GND), U25.8 (GND), U25.9 (GND), U26.2 (GND), U26.3 (GND), U26.4 (GND), U26.7 (GND), U26.8 (GND), U26.9 (GND), J1.1 (Pin_1), J3.4 (Pin_4), J5.4 (Pin_4)
- net I2C1_SCL: now also J3.5 (Pin_5)
- net I2C1_SDA: now also J3.6 (Pin_6)
- net I2C2_SCL: now also J5.5 (Pin_5)
- net I2C2_SDA: now also J5.6 (Pin_6)
- net LED_L: now also J5.3 (Pin_3)
- net LED_R: now also J3.3 (Pin_3)
- net photo_L_1: now also J1.8 (Pin_8)
- net photo_L_2: now also J1.7 (Pin_7)
- net photo_L_3: now also J1.6 (Pin_6)
- net photo_L_4: now also J1.5 (Pin_5)
- net photo_L_5: now also J1.4 (Pin_4)
- net photo_L_6: now also J1.3 (Pin_3)
- net photo_L_7: now also J1.2 (Pin_2)
- net photo_R_1: now also J1.11 (Pin_11)
- net photo_R_2: now also J1.12 (Pin_12)
- net photo_R_3: now also J1.13 (Pin_13)
- net photo_R_4: now also J1.14 (Pin_14)
- net photo_R_5: now also J1.15 (Pin_15)
- net photo_R_6: now also J1.16 (Pin_16)
- net photo_R_7: now also J1.17 (Pin_17)
- net photo_center: now also J1.9 (Pin_9)
- net photo_front: now also J1.10 (Pin_10)
- net +5V renamed 5V_LED
- net 5V_LED: now also J3.2 (Pin_2), J5.2 (Pin_2)
- new net SENSER_3V3: C3.1, C6.1, J3.1 (Pin_1), J5.1 (Pin_1), U25.1 (VDD), U26.1 (VDD)
- no-connect marks 23 -> 2
Other:
- moved on the sheet: C3, C6, D1, D2, D4, D5, D6, D8, R1, R10, R11, R12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
