File: 04-line/04-line.kicad_pcb (KiCad board)
At the start: 2 copper layers, 72 parts, among them J2 VL53L0X, J3 ToMAIN, J4 WRITER CONN, U24 STM32F446RETx

Commit message: line...
Parts:
- added C1: 100n, Capacitor_SMD:C_0805_2012Metric, B.Cu at (55.9, 128.6)
- added C10: 100u, Capacitor_SMD:C_0805_2012Metric, B.Cu at (104.5, 147.3)
- added C2: 4.7u, Capacitor_SMD:C_0805_2012Metric, B.Cu at (87.6, 125.7)
- added C3: 0.1u, Capacitor_SMD:C_0805_2012Metric, B.Cu at (73.7, 76.2)
- added C4: 1u, Capacitor_SMD:C_0805_2012Metric, B.Cu at (76.2, 116.8)
- added C5: 1u, Capacitor_SMD:C_0805_2012Metric, B.Cu at (96.5, 132.1)
- added C6: 0.1u, Capacitor_SMD:C_0805_2012Metric, B.Cu at (93.0, 76.2)
- added C7: 10u, Capacitor_SMD:C_0805_2012Metric, B.Cu at (107.0, 152.4)
- added C8: 10u, Capacitor_SMD:C_0805_2012Metric, B.Cu at (118.1, 152.4)
- added C9: 0.33u, Capacitor_SMD:C_0805_2012Metric, B.Cu at (113.0, 152.4)
- added R38: 100k, Resistor_SMD:R_0805_2012Metric, B.Cu at (76.2, 120.7)
- added R39: 100k, Resistor_SMD:R_0805_2012Metric, B.Cu at (92.4, 132.1)
- D1, D2, D3, D4, J2, R1, R10, R11, R12, R13, R14, R15, R16, R17, R18, R19, R2, R20, R21, R22, R23, R24, R25, R26, R27, R28, R29, R3, R30, R31, R32, R33, R34, R35, R36, R4, R5, R6, R7, R8, R9, U1, U10, U11, U12, U13, U14, U15, U16, U17, U18, U19, U2, U20, U21, U22, U23, U24, U25, U26, U27, U28, U3, U4, U5, U6, U7, U8, U9: moved to B.Cu
- moved R37 125.3 mm to (63.5, 148.6)
- moved U27 110.6 mm to (113.0, 143.5), turned to 180 degrees
- moved U21 87.7 mm to (110.4, 114.3)
- moved J3 81.3 mm to (83.8, 149.9), turned to 180 degrees
- moved U1 79.9 mm to (49.6, 114.3)
- moved U23 79.8 mm to (96.5, 114.3)
- moved U11 79.6 mm to (67.4, 114.3)
- moved U22 79.6 mm to (83.9, 114.3)
- moved U28 69.3 mm to (96.3, 145.6), turned to 90 degrees
- moved R10 69.1 mm to (43.2, 89.3), turned to -90 degrees
- moved U12 63.8 mm to (114.0, 97.0), turned to -90 degrees
- moved R11 62.9 mm to (48.9, 89.5), turned to -90 degrees
- moved J4 62.2 mm to (55.9, 143.5)
- moved R12 57.0 mm to (54.0, 89.5), turned to -90 degrees
- moved U2 56.3 mm to (42.9, 97.0), turned to -90 degrees
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
Commit message: ラインセンサ完成
Parts:
- removed R27: 105, Resistor_SMD:R_0603_1608Metric
- removed R35, R36: 1k, Resistor_SMD:R_1206_3216Metric
- removed R38, R39: 100k, Resistor_SMD:R_0805_2012Metric
- removed U1, U11, U21, U22, U23: ~, Package_SO:SOIC-14_3.9x8.7mm_P1.27mm
- removed U19, U20: ~, Akiduki:LBR127HLD
- added C11: 100n, Capacitor_SMD:C_0402_1005Metric, B.Cu at (99.1, 125.7)
- added C12: 100n, Capacitor_SMD:C_0402_1005Metric, B.Cu at (92.7, 120.7)
- added C13: 100n, Capacitor_SMD:C_0402_1005Metric, B.Cu at (87.6, 138.4)
- added C14: 4.7u, Capacitor_SMD:C_0402_1005Metric, B.Cu at (78.7, 133.3)
- added C15: 100n, Capacitor_SMD:C_0402_1005Metric, B.Cu at (81.3, 121.9)
- added C16: 1u, Capacitor_SMD:C_0402_1005Metric, B.Cu at (81.3, 120.7)
- added D5: WS2812B, LED_SMD:LED_WS2812B_PLCC4_5.0x5.0mm_P3.2mm, B.Cu at (69.4, 97.0)
- added D6: WS2812B, LED_SMD:LED_WS2812B_PLCC4_5.0x5.0mm_P3.2mm, B.Cu at (77.4, 90.0)
- added D7: WS2812B, LED_SMD:LED_WS2812B_PLCC4_5.0x5.0mm_P3.2mm, B.Cu at (69.4, 83.0)
- added D8: WS2812B, LED_SMD:LED_WS2812B_PLCC4_5.0x5.0mm_P3.2mm, B.Cu at (61.4, 90.0)
- added FB1: FerriteBead, Resistor_SMD:R_0805_2012Metric, B.Cu at (77.5, 121.9)
- added G***: LOGO, logo:jlcpcb_logo_big, F.Cu at (69.6, 97.3)
- added G***: LOGO, logo:tuton_logo, F.Cu at (99.3, 96.3)
- added J1: ST-LINK, Connector_PinHeader_2.54mm:PinHeader_1x04_P2.54mm_Vertical, F.Cu at (52.1, 132.1)
- added J5: SSD1306, Connector_PinHeader_2.54mm:PinHeader_1x04_P2.54mm_Vertical, F.Cu at (97.8, 76.2)
- C1, C2: footprint Capacitor_SMD:C_0805_2012Metric -> Capacitor_SMD:C_0402_1005Metric
- C10: footprint Capacitor_SMD:C_0805_2012Metric -> Capacitor_SMD:C_1206_3216Metric
- C3, C6: value 0.1u -> 100n; footprint Capacitor_SMD:C_0805_2012Metric -> Capacitor_SMD:C_0402_1005Metric
- C4, C5: value 1u -> 100n; footprint Capacitor_SMD:C_0805_2012Metric -> Capacitor_SMD:C_0402_1005Metric
- C7, C8: footprint Capacitor_SMD:C_0805_2012Metric -> Capacitor_SMD:C_0603_1608Metric
- R26: value 105 -> 10k
- R37: footprint Resistor_SMD:R_0805_2012Metric -> Resistor_SMD:R_0603_1608Metric; moved to B.Cu
- moved R26 56.4 mm to (101.6, 120.7), turned to 0 degrees
- moved D2 45.8 mm to (109.4, 90.0), turned to -90 degrees
- moved R10 45.0 mm to (78.7, 116.8), turned to 90 degrees
- moved R34 44.3 mm to (119.4, 116.8), turned to 90 degrees
- moved U18 39.6 mm to (121.0, 110.0), turned to 90 degrees
- moved U2 39.6 mm to (80.3, 110.0), turned to 90 degrees
- moved R16 37.7 mm to (48.3, 116.8), turned to 90 degrees
- moved R28 37.7 mm to (88.9, 116.8), turned to 90 degrees
- moved R1 37.0 mm to (80.8, 102.9), turned to 90 degrees
- moved R25 37.0 mm to (121.5, 102.9), turned to 90 degrees
- moved R33 36.9 mm to (114.3, 116.8), turned to 90 degrees
- moved R11 36.9 mm to (73.7, 116.8), turned to 90 degrees
- moved U26 35.4 mm to (101.4, 90.0)
- moved D3 32.7 mm to (101.4, 83.0)
- moved R15 31.6 mm to (53.3, 116.8), turned to 90 degrees
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Connections:
- C4 pad 1: Ag_Com -> GND
- C4 pad 2: GND -> +3V3
- C5 pad 1: B_W_Com -> GND
- C5 pad 2: GND -> +3V3
- D1 pad 4: Net-(D1-DIN) -> LED_L
- J2 pad 3: I2C1_SCL -> I2C3_SCL
- J2 pad 4: I2C1_SDA -> I2C3_SDA
- J3 pad 3: UART2_RX -> UART3_RX
- J3 pad 4: UART2_TX -> UART3_TX
- R26 pad 1: Net-(U19-Cathode) -> Net-(U24-PB2)
- U24 pad 10: unconnected-(U24-PC2-Pad10) -> photo_L_5
- U24 pad 11: unconnected-(U24-PC3-Pad11) -> photo_L_4
- U24 pad 13: +3V3 -> Net-(U24-VDDA)
- U24 pad 14: unconnected-(U24-PA0-Pad14) -> photo_L_3
- U24 pad 15: unconnected-(U24-PA1-Pad15) -> photo_L_2
- U24 pad 16: UART2_TX -> photo_L_1
- U24 pad 17: UART2_RX -> photo_front
- U24 pad 20: unconnected-(U24-PA4-Pad20) -> photo_center
- U24 pad 21: unconnected-(U24-PA5-Pad21) -> photo_R_1
- U24 pad 22: Net-(U24-PA6) -> photo_R_2
- U24 pad 23: unconnected-(U24-PA7-Pad23) -> photo_R_3
- U24 pad 24: unconnected-(U24-PC4-Pad24) -> photo_R_4
- U24 pad 25: unconnected-(U24-PC5-Pad25) -> photo_R_5
- U24 pad 26: unconnected-(U24-PB0-Pad26) -> photo_R_6
- U24 pad 27: unconnected-(U24-PB1-Pad27) -> photo_R_7
- U24 pad 28: unconnected-(U24-PB2-Pad28) -> Net-(U24-PB2)
- U24 pad 3: unconnected-(U24-PC14-Pad3) -> LED_R
- U24 pad 33: Net-(D1-DIN) -> unconnected-(U24-PB12-Pad33)
- U24 pad 34: RR_OUT -> unconnected-(U24-PB13-Pad34)
- U24 pad 35: LL_OUT -> unconnected-(U24-PB14-Pad35)
- U24 pad 36: R_1_OUT -> unconnected-(U24-PB15-Pad36)
- U24 pad 37: R_2_OUT -> unconnected-(U24-PC6-Pad37)
- U24 pad 38: R_3_OUT -> unconnected-(U24-PC7-Pad38)
- U24 pad 39: R_4_OUT -> unconnected-(U24-PC8-Pad39)
- U24 pad 4: unconnected-(U24-PC15-Pad4) -> LED_L
- U24 pad 40: R_5_OUT -> I2C3_SDA
- U24 pad 41: Net-(U24-PA8) -> I2C3_SCL
- U24 pad 44: R_6_OUT -> unconnected-(U24-PA11-Pad44)
- U24 pad 45: R_7_OUT -> unconnected-(U24-PA12-Pad45)
- U24 pad 46: front_OUT -> SWDIO
- U24 pad 49: center_OUT -> SWCLK
- U24 pad 50: L_7_OUT -> unconnected-(U24-PA15-Pad50)
- U24 pad 51: L_6_OUT -> UART3_TX
- U24 pad 52: L_5_OUT -> UART3_RX
- U24 pad 54: L_4_OUT -> unconnected-(U24-PD2-Pad54)
- U24 pad 55: L_3_OUT -> unconnected-(U24-PB3-Pad55)
- U24 pad 56: L_2_OUT -> unconnected-(U24-PB4-Pad56)
- U24 pad 57: L_1_OUT -> unconnected-(U24-PB5-Pad57)
- U24 pad 8: unconnected-(U24-PC0-Pad8) -> photo_L_7
- U24 pad 9: unconnected-(U24-PC1-Pad9) -> photo_L_6
- U25 pad 2: (no net) -> GND
- U25 pad 3: (no net) -> GND
- U25 pad 4: (no net) -> GND
- U25 pad 7: (no net) -> GND
- U25 pad 8: (no net) -> GND
- U25 pad 9: (no net) -> GND
- U26 pad 2: (no net) -> GND
- U26 pad 3: (no net) -> GND
- U26 pad 4: (no net) -> GND
- U26 pad 7: (no net) -> GND
- U26 pad 8: (no net) -> GND
- U26 pad 9: (no net) -> GND
Routing:
- net +3V3: track 0.00 -> 348.0 mm, vias 0 -> 2
- net GND: track 0.00 -> 162.0 mm, vias 0 -> 77
- net +5V: track 0.00 -> 151.3 mm
- net I2C3_SCL: track 0.00 -> 129.4 mm, vias 0 -> 1
- net I2C3_SDA: track 0.00 -> 127.9 mm, vias 0 -> 1
- net I2C2_SDA: track 0.00 -> 116.7 mm, vias 0 -> 2
- net I2C1_SDA: track 0.00 -> 87.6 mm, vias 0 -> 4
- net I2C1_SCL: track 0.00 -> 85.2 mm, vias 0 -> 4
- net LED_L: track 0.00 -> 82.3 mm, vias 0 -> 2
- net VDD: track 0.00 -> 76.1 mm
- net I2C2_SCL: track 0.00 -> 61.4 mm, vias 0 -> 4
- net UART1_TX: track 0.00 -> 61.2 mm, vias 0 -> 1
- net SWDIO: track 0.00 -> 53.6 mm, vias 0 -> 2
- net UART1_RX: track 0.00 -> 53.1 mm, vias 0 -> 1
- net photo_L_7: track 0.00 -> 45.8 mm, vias 0 -> 3
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- added copper zone on B.Cu, net GND
- added copper zone on F.Cu, net GND
Other:
- board outline added: 80 x 75 mm
- board text added: "04-LINE ver.1"
- board text added: "1"
- board text added: "3V3"
- board text added: "3V3 REG"
- board text added: "5V REG"
- board text added: "BOOT0"
- board text added: "GND"
- board text added: "JLCJLCJLCJLC"
- board text added: "NRST"
- board text added: "RX"
- board text added: "RX→"
- board text added: "SCL"
- board text added: "SDA"
- board text added: "SSD1306"
- board text added: "SWCLK"
- board text added: "SWDIO"
- board text added: "TX"
- board text added: "TX←"
- board text added: "VDD"
- board text added: "VL53L0X"
- board text added: "↓"

Commit message: 前けずった
Parts:
- removed D3, D7: WS2812B, LED_SMD:LED_WS2812B_PLCC4_5.0x5.0mm_P3.2mm
- removed J2: VL53L0X, Connector_PinHeader_2.54mm:PinHeader_1x04_P2.54mm_Vertical
- removed J5: SSD1306, Connector_PinHeader_2.54mm:PinHeader_1x04_P2.54mm_Vertical
- moved C3 2.03 mm to (77.5, 84.6)
- moved G*** 0.80 mm to (99.1, 97.0)
- moved G*** 0.76 mm to (69.6, 98.0)
Connections:
- D4 pad 4: Net-(D3-DOUT) -> Net-(D2-DOUT)
- D8 pad 4: Net-(D7-DOUT) -> Net-(D6-DOUT)
Routing:
- net I2C3_SCL: track 129.4 -> 0.00 mm, vias 1 -> 0
- net I2C3_SDA: track 127.9 -> 0.00 mm, vias 1 -> 0
- net +3V3: track 348.0 -> 307.9 mm
- net GND: track 162.0 -> 145.7 mm, vias 77 -> 76
- net Net-(D6-DOUT): track 8.40 -> 20.4 mm
- net Net-(D3-DOUT): track 10.3 -> 0.00 mm, vias 2 -> 0
- net Net-(D7-DOUT): track 7.82 -> 0.00 mm
- net +5V: track 151.3 -> 147.4 mm
- net Net-(D2-DOUT): track 16.3 -> 19.5 mm
Other:
- board size 80 x 75 mm -> 80 x 65 mm
- board text removed: "SCL"
- board text removed: "SDA"
- board text removed: "SSD1306"
- board text removed: "VL53L0X"

Commit message: いっぱい増えた
Parts:
- removed C1, C11, C12, C13, C15, C4, C5: 100n, Capacitor_SMD:C_0402_1005Metric
- removed C10: 100u, Capacitor_SMD:C_1206_3216Metric
- removed C14, C2: 4.7u, Capacitor_SMD:C_0402_1005Metric
- removed C16: 1u, Capacitor_SMD:C_0402_1005Metric
- removed C7, C8: 10u, Capacitor_SMD:C_0603_1608Metric
- removed C9: 0.33u, Capacitor_SMD:C_0805_2012Metric
- removed FB1: FerriteBead, Resistor_SMD:R_0805_2012Metric
- removed J4: WRITER CONN, Connector_PinHeader_2.54mm:PinHeader_2x04_P2.54mm_Vertical
- removed R26, R37: 10k, Resistor_SMD:R_0603_1608Metric
- removed U24: STM32F446RETx, Package_QFP:LQFP-64_10x10mm_P0.5mm
- removed U27: ~, Package_TO_SOT_SMD:SOT-223-6
- removed U28: ~, Package_TO_SOT_SMD:TO-252-3_TabPin2
- added J2: CS_R, Connector_PinHeader_2.54mm:PinHeader_2x03_P2.54mm_Vertical, B.Cu at (68.6, 87.6)
- added REF**: MountingHole_3.2mm_M3, MountingHole:MountingHole_3.2mm_M3, F.Cu at (67.6, 78.6)
- added REF**: MountingHole_3.2mm_M3, MountingHole:MountingHole_3.2mm_M3, F.Cu at (135.6, 78.6)
- added REF**: MountingHole_3.2mm_M3, MountingHole:MountingHole_3.2mm_M3, F.Cu at (119.6, 121.6)
- added REF**: MountingHole_3.2mm_M3, MountingHole:MountingHole_3.2mm_M3, F.Cu at (83.6, 121.6)
- C3, C6, D1, D2, D4, D5, D6, D8, U10, U12, U13, U14, U15, U16, U17, U18, U2, U25, U26, U3, U4, U5, U6, U7, U8, U9: moved to F.Cu
- G*** (x2): moved to B.Cu
- J1: value ST-LINK -> Conn_01x18; footprint Connector_PinHeader_2.54mm:PinHeader_1x04_P2.54mm_Vertical -> Connector_PinHeader_2.54mm:PinHeader_1x18_P2.54mm_Vertical; moved to B.Cu
- J3: value ToMAIN -> CS_L; footprint Connector_JST:JST_XH_B4B-XH-A_1x04_P2.50mm_Vertical -> Connector_PinHeader_2.54mm:PinHeader_2x03_P2.54mm_Vertical; moved to B.Cu
- R1, R19, R2, R20, R21, R22, R23, R24, R25, R3, R4, R5, R6, R7, R8, R9: value 105 -> 120; moved to F.Cu
- R10, R11, R12, R13, R14, R15, R16, R17, R18, R28, R29, R30, R31, R32, R33, R34: footprint Resistor_SMD:R_1206_3216Metric -> Resistor_SMD:R_0603_1608Metric; moved to F.Cu
- moved J3 81.6 mm to (129.5, 87.6), turned to -90 degrees
- moved C3 50.9 mm to (128.3, 81.3), turned to -90 degrees
- moved U25 48.2 mm to (116.8, 81.4), turned to 0 degrees
- moved G*** 42.3 mm to (111.3, 90.7), turned to 180 degrees
- moved J1 36.1 mm to (80.0, 109.2), turned to -90 degrees
- moved C6 35.7 mm to (74.9, 80.8), turned to -90 degrees
- moved R16 34.5 mm to (82.5, 113.0)
- moved R15 32.0 mm to (85.1, 113.0)
- moved R14 29.5 mm to (87.6, 113.0)
- moved R13 26.9 mm to (90.2, 113.0)
- moved R12 24.4 mm to (92.7, 113.0)
- moved R18 24.4 mm to (102.9, 113.0)
- moved R9 22.2 mm to (105.4, 88.9), turned to -90 degrees
- moved R11 21.9 mm to (95.2, 113.0)
- moved R10 19.4 mm to (97.8, 113.0)
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Connections:
- C3 pad 1: +3V3 -> SENSER_3V3
- C6 pad 1: +3V3 -> SENSER_3V3
- D1 pad 1: +5V -> 5V_LED
- D2 pad 1: +5V -> 5V_LED
- D4 pad 1: +5V -> 5V_LED
- D5 pad 1: +5V -> 5V_LED
- D6 pad 1: +5V -> 5V_LED
- D8 pad 1: +5V -> 5V_LED
- J1 pad 1: SWCLK -> GND
- J1 pad 2: SWDIO -> photo_L_7
- J1 pad 3: NRST -> photo_L_6
- J1 pad 4: GND -> photo_L_5
- J3 pad 1: VDD -> SENSER_3V3
- J3 pad 2: GND -> 5V_LED
- J3 pad 3: UART3_RX -> LED_L
- J3 pad 4: UART3_TX -> GND
- U25 pad 1: +3V3 -> SENSER_3V3
- U26 pad 1: +3V3 -> SENSER_3V3
Routing:
- net +5V: track 147.4 -> 0.00 mm
- net +3V3: track 307.9 -> 181.0 mm, vias 2 -> 0
- net 5V_LED: track 0.00 -> 98.5 mm
- net I2C2_SDA: track 116.7 -> 25.4 mm, vias 2 -> 1
- net GND: track 145.7 -> 60.0 mm, vias 76 -> 29
- net SENSER_3V3: track 0.00 -> 82.3 mm, vias 0 -> 4
- net VDD: track 76.1 -> 0.00 mm
- net I2C1_SCL: track 85.2 -> 16.8 mm, vias 4 -> 0
- net LED_L: track 82.3 -> 14.0 mm, vias 2 -> 0
- net I2C1_SDA: track 87.6 -> 23.3 mm, vias 4 -> 0
- net UART1_TX: track 61.2 -> 0.00 mm, vias 1 -> 0
- net SWDIO: track 53.6 -> 0.00 mm, vias 2 -> 0
- net UART1_RX: track 53.1 -> 0.00 mm, vias 1 -> 0
- net I2C2_SCL: track 61.4 -> 17.8 mm, vias 4 -> 1
- net SWCLK: track 42.9 -> 0.00 mm, vias 2 -> 0
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Other:
- board size 80 x 65 mm -> 80 x 52 mm
- board text removed: "04-LINE ver.1"
- board text removed: "1"
- board text removed: "3V3"
- board text removed: "3V3 REG"
- board text removed: "5V REG"
- board text removed: "BOOT0"
- board text removed: "GND"
- board text removed: "JLCJLCJLCJLC"
- board text removed: "NRST"
- board text removed: "RX"
- board text removed: "RX→"
- board text removed: "SWCLK"
- board text removed: "SWDIO"
- board text removed: "TX"
- board text removed: "TX←"
- board text removed: "VDD"
- board text removed: "↓"

Commit message: pdf
Parts:
- added G***: LOGO, logo:st_logo_middle, F.Cu at (132.7, 118.1)
- added G***: LOGO, logo:jlcpcb_logo, F.Cu at (71.1, 117.5)
- added G***: LOGO, logo:st_logo_middle, B.Cu at (102.2, 120.0)
Other:
- board text added: "04-LINE ver.2"
- board text added: "3V3"
- board text added: "5V"
- board text added: "GND"
- board text added: "LED_R"
- board text added: "RCJ 2025 tuton"
- board text added: "SCL"
- board text added: "SDA"
