File: 06_WRITER/06_WRITER.kicad_sch (KiCad schematic)
At the start: 13 parts, among them J1 USB_C_Receptacle_USB2.0, J2 Conn_02x04_Counter_Clockwise, SW1 NRST, SW2 BOOT0, U1 CH340E

Commit message: いっぱい増えた
Parts:
- C1, C2: LCSC C38141 -> C49678
- R1, R2: LCSC C2828689 -> C27834
Changed lines of the file:
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@@
       (effects (font (size 1.27 1.27)) hide)
     )
-    (property "LCSC" "C2828689" (at 72.39 49.53 0)
+    (property "LCSC" "C27834" (at 72.39 49.53 0)
       (effects (font (size 1.27 1.27)) hide)
     )
@@
       (effects (font (size 1.27 1.27)) hide)
     )
-    (property "LCSC" "C38141" (at 60.96 97.155 0)
+    (property "LCSC" "C49678" (at 60.96 97.155 0)
       (effects (font (size 1.27 1.27)) hide)
     )
@@
       (effects (font (size 1.27 1.27)) hide)
     )
-    (property "LCSC" "C38141" (at 46.355 97.155 0)
+    (property "LCSC" "C49678" (at 46.355 97.155 0)
       (effects (font (size 1.27 1.27)) hide)
     )
@@
       (effects (font (size 1.27 1.27)) hide)
     )
-    (property "LCSC" "C2828689" (at 80.645 49.53 0)
+    (property "LCSC" "C27834" (at 80.645 49.53 0)
       (effects (font (size 1.27 1.27)) hide)
     )
