File: 08-REG_mod/08-REG_mod.kicad_pcb (KiCad board)
At the start: 2 copper layers, 19.7 x 26.7 mm, 12 parts, among them J1 Conn_01x05, U1 TPS5430DDA

Commit message: パワー
Parts:
- added G***: LOGO, logo:st_logo, B.Cu at (106.7, 61.6)
- moved G*** 3.18 mm to (111.8, 61.6)
Other:
- board text added: "DCDC by tuton"
- board text removed: "えすてぃい"
- board text removed: "このDCDCは燃えないよ"
