File: 08-REG_mod/08-REG_mod.kicad_sch (KiCad schematic)
At the start: 10 parts, among them J1 Conn_01x05, U1 TPS5430DDA

Commit message: pdf
Other:
- note removed: "入力電圧範囲 10.5~12.6V 出力電圧 7.2V 出力電圧定格 1.5A 動作周波数 500kHz"
Changed lines of the file:
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@@
     (stroke (width 0) (type default))
   )
-  (text "入力電圧範囲　10.5~12.6V\n出力電圧　7.2V\n出力電圧定格　1.5A\n動作周波数　500kHz\n"
-    (at 48.895 96.52 0)
+  (text "2.04k\n" (at 161.29 93.98 0)
     (effects (font (size 1.27 1.27)) (justify left bottom))
   )
-  (text "2.04k\n" (at 48.895 102.235 0)
-    (effects (font (size 1.27 1.27)) (justify left bottom))
-  )
