File: 04-line_sub/04-line_sub.kicad_pcb (KiCad board)
At the start: 2 copper layers, 71.1 x 35.6 mm, 25 parts, among them J1 Conn_01x06, J2 WRITER CONN, J3 CS_R, J4 Conn_01x18, J5 CS_L, U1 STM32F446RETx

Commit message: pdf
Parts:
- added G***: LOGO, logo:tuton_logo_small, F.Cu at (123.2, 95.2)
- added G***: LOGO, logo:jlcpcb_logo, F.Cu at (119.4, 90.2)
- added G***: LOGO, logo:st_logo, F.Cu at (112.4, 95.2)
- added G***: LOGO, logo:tuton_logo_small, B.Cu at (101.6, 99.7)
- added G***: LOGO, logo:jlcpcb_logo, B.Cu at (115.6, 100.3)
- added G***: LOGO, logo:st_logo, B.Cu at (89.5, 101.0)
Other:
- board text added: "04-LINE ver.2"
- board text added: "1"
- board text added: "3V3L"
- board text added: "RCJ 2025 tuton"
- board text removed: "3V3lbr"
- board text removed: "5V LED"
