File: 04-line_sub/04-line_sub.kicad_sch (KiCad schematic)
At the start: 25 parts, among them J1 Conn_01x06, J2 WRITER CONN, J3 CS_R, J4 Conn_01x18, J5 CS_L, U1 STM32F446RETx

Commit message: pdf
Other:
- title: (none) -> 04-line_sub
Changed lines of the file:
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@@
 (kicad_sch (version 20230121) (generator eeschema)
   (paper "A4")
+  (title_block
+    (title "04-line_sub")
+    (date "2024-06-27")
+  )
   (junction (at 90.805 59.055) (diameter 0) (color 0 0 0 0)
   )
