File: 05-PWR/05-PWR.kicad_pcb (KiCad board)
At the start: 2 copper layers, 160 x 60 mm, 13 parts, among them J1 VDD_IN, J2 GND, J3 VDD_OUT, J4 GND, J5 Ammeter, J6 Voltmeter, J7 Conn_01x04, SW1 SW_DIP_x01, SW2 SW_Push, SW3 SW_SPDT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

Commit message: 全国行きたかった
Parts:
- removed SW1: SW_DIP_x01, Connector_PinHeader_2.54mm:PinHeader_1x02_P2.54mm_Vertical
- added G***: LOGO, logo:tuton_logo_big, F.Cu at (116.8, 83.8)
- added G***: LOGO, logo:jlcpcb_logo_big, F.Cu at (116.8, 101.6)
- added J10: AMMETER_V, Connector_PinHeader_2.54mm:PinHeader_1x01_P2.54mm_Vertical, F.Cu at (134.6, 121.9)
- added J11: AMMETER_G, Connector_PinHeader_2.54mm:PinHeader_1x01_P2.54mm_Vertical, F.Cu at (134.6, 106.7)
- added J12: AMMETER_G, Connector_PinHeader_2.54mm:PinHeader_1x01_P2.54mm_Vertical, F.Cu at (134.6, 114.3)
- added J8: VOLTMETER_V, Connector_PinHeader_2.54mm:PinHeader_1x01_P2.54mm_Vertical, F.Cu at (179.1, 106.7)
- added J9: VOLTMETER_G, Connector_PinHeader_2.54mm:PinHeader_1x01_P2.54mm_Vertical, F.Cu at (179.1, 90.2)
- J5: value Ammeter -> SW_VI; footprint Connector_PinSocket_2.54mm:PinSocket_1x03_P2.54mm_Vertical -> Connector_PinHeader_2.54mm:PinHeader_1x01_P2.54mm_Vertical
- J6: value Voltmeter -> SW_VO; footprint Connector_PinSocket_2.54mm:PinSocket_1x02_P2.54mm_Vertical -> Connector_PinHeader_2.54mm:PinHeader_1x01_P2.54mm_Vertical
- moved J5 38.9 mm to (189.2, 98.8), turned to 0 degrees
- moved J6 26.4 mm to (189.2, 106.7), turned to 0 degrees
- moved J1 5.22 mm to (185.6, 121.9)
- moved J4 4.24 mm to (185.4, 76.2)
- moved SW2 1.66 mm to (60.8, 95.2)
- moved SW4 1.66 mm to (60.6, 105.7)
- moved SW5 1.66 mm to (60.8, 115.6)
- moved F1 1.11 mm to (203.2, 121.9)
Connections:
- F1 pad 2: Net-(F1-Pad2) -> Net-(J5-Pin_1)
- J3 pad 1: Net-(J3-Pin_1) -> Net-(J10-Pin_1)
- J5 pad 1: Net-(J3-Pin_1) -> Net-(J5-Pin_1)
- J6 pad 1: Net-(J3-Pin_1) -> Net-(J10-Pin_1)
Routing:
- net Net-(J10-Pin_1): track 0.00 -> 110.9 mm
- net Net-(J7-Pin_3): track 0.00 -> 37.9 mm
- net Net-(J7-Pin_2): track 0.00 -> 32.1 mm
- net Net-(J7-Pin_1): track 0.00 -> 31.9 mm
- net Net-(J1-Pin_1): track 0.00 -> 24.4 mm
- net Net-(J7-Pin_4): track 0.00 -> 21.4 mm
- net Net-(J5-Pin_1): track 0.00 -> 20.7 mm
Other:
- outline, holes or cut-outs redrawn
- board text added: "AM_A+"
- board text added: "AM_COM"
- board text added: "AM_V+"
- board text added: "FUSE"
- board text added: "GND"
- board text added: "POWER BOARD V1"
- board text added: "PWR_SW"
- board text added: "SIG"
- board text added: "SW1"
- board text added: "SW2"
- board text added: "SW3"
- board text added: "TOGGLE"
- board text added: "VDD_IN"
- board text added: "VDD_OUT"
- board text added: "VM+"
- board text added: "VM-"
- board text added: "x"

Commit message: がんばる
Parts:
- removed G***: LOGO, logo:tuton_logo_big
- removed G***: LOGO, logo:jlcpcb_logo_big
- J7: moved to F.Cu
- moved J6 113.9 mm to (88.5, 53.6)
- moved SW2 113.3 mm to (171.9, 73.0)
- moved J5 112.4 mm to (88.5, 48.9)
- moved J2 106.6 mm to (187.5, 116.8)
- moved J8 102.7 mm to (88.5, 58.2)
- moved J9 94.6 mm to (88.5, 62.9)
- moved J4 90.9 mm to (103.5, 115.6)
- moved SW5 84.3 mm to (141.5, 91.1)
- moved J10 83.9 mm to (93.2, 48.9)
- moved F1 72.8 mm to (160.7, 62.9)
- moved J12 69.7 mm to (93.2, 58.2)
- moved SW4 69.1 mm to (128.2, 91.1)
- moved J11 67.4 mm to (93.2, 53.6)
- moved SW3 67.1 mm to (155.6, 86.3)
- moved J7 54.9 mm to (130.3, 70.5)
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Routing:
- net Net-(J10-Pin_1): track 110.9 -> 0.00 mm
- net Net-(J7-Pin_3): track 37.9 -> 0.00 mm
- net Net-(J7-Pin_2): track 32.1 -> 0.00 mm
- net Net-(J7-Pin_1): track 31.9 -> 0.00 mm
- net Net-(J1-Pin_1): track 24.4 -> 0.00 mm
- net Net-(J7-Pin_4): track 21.4 -> 0.00 mm
- net Net-(J5-Pin_1): track 20.7 -> 0.00 mm
Other:
- board outline removed
- board text removed: "AM_A+"
- board text removed: "AM_COM"
- board text removed: "AM_V+"
- board text removed: "FUSE"
- board text removed: "GND"
- board text removed: "POWER BOARD V1"
- board text removed: "PWR_SW"
- board text removed: "SIG"
- board text removed: "SW1"
- board text removed: "SW2"
- board text removed: "SW3"
- board text removed: "TOGGLE"
- board text removed: "VDD_IN"
- board text removed: "VDD_OUT"
- board text removed: "VM+"
- board text removed: "VM-"
- board text removed: "x"

Commit message: いっぱい増えた
Parts:
- removed F1: Fuse, Fuse:Fuseholder_Clip-5x20mm_Keystone_3517_Inline_P23.11x6.76mm_D1.70mm_Horizontal
- removed J11, J12: AMMETER_G, Connector_PinHeader_2.54mm:PinHeader_1x01_P2.54mm_Vertical
- removed SW2, SW4, SW5: SW_Push, Button_Switch_THT:SW_PUSH_6mm
- removed SW3: SW_SPDT, Connector_PinHeader_2.54mm:PinHeader_1x03_P2.54mm_Vertical
- added C1: 22uF, Capacitor_SMD:C_0805_2012Metric, F.Cu at (52.1, 43.3)
- added C2: 10uF, Capacitor_SMD:C_0805_2012Metric, F.Cu at (52.1, 46.4)
- added C3: 22uF, Capacitor_SMD:C_0805_2012Metric, F.Cu at (52.1, 49.4)
- added C4: 10uF, Capacitor_SMD:C_0805_2012Metric, F.Cu at (52.1, 52.4)
- added Q1: Q_PMOS_GDS, Package_TO_SOT_THT:TO-251-3_Vertical, F.Cu at (53.0, 72.1)
- added R1: 1k, Resistor_SMD:R_0603_1608Metric, F.Cu at (79.5, 26.8)
- added R2: 330, Resistor_SMD:R_0603_1608Metric, F.Cu at (79.5, 29.3)
- added R3: 10, Resistor_SMD:R_0603_1608Metric, F.Cu at (79.5, 31.8)
- added R4: 1.2k, Resistor_SMD:R_0603_1608Metric, F.Cu at (79.5, 34.3)
- added R5: 1.5k, Resistor_SMD:R_0603_1608Metric, F.Cu at (79.5, 36.8)
- added R6: 680, Resistor_SMD:R_0603_1608Metric, F.Cu at (79.5, 39.3)
- added R7: 10k, Resistor_SMD:R_0603_1608Metric, F.Cu at (79.5, 41.8)
- added R8: 1.2k, Resistor_SMD:R_0603_1608Metric, F.Cu at (79.5, 44.3)
- added R9: 10k, Resistor_SMD:R_0603_1608Metric, F.Cu at (79.5, 46.9)
- added REF**: voltmeter, Akiduki:Voltmeter, F.Cu at (229.2, 74.9)
- added RV1: R_Trim, Potentiometer_THT:Potentiometer_Bourns_3296W_Vertical, F.Cu at (143.5, 59.1)
- added RV2: R_Trim, Potentiometer_THT:Potentiometer_Bourns_3296W_Vertical, F.Cu at (144.8, 70.5)
- added RV3: R_Trim, Potentiometer_THT:Potentiometer_Bourns_3296W_Vertical, F.Cu at (144.8, 76.9)
- added SW1: SW_SPST, Akiduki:DS-850K-S-ON, F.Cu at (240.0, 52.7)
- added U1: ~, Connector_PinHeader_2.54mm:PinHeader_1x05_P2.54mm_Vertical, F.Cu at (37.5, 65.4)
- added U2: ~, Connector_PinHeader_2.54mm:PinHeader_1x05_P2.54mm_Vertical, F.Cu at (37.5, 76.8)
- added U3: ~, Akiduki:OKL-T6-W12N-C, F.Cu at (169.2, 58.6)
- added U4: ~, Akiduki:OKL-T6-W12N-C, F.Cu at (160.3, 43.4)
- J1: value VDD_IN -> Battery; footprint MountingHole:MountingHole_3.2mm_M3_Pad_Via -> Connector_Wire:SolderWire-2sqmm_1x02_P7.8mm_D2mm_OD3.9mm
- J10: value AMMETER_V -> 5V ToMAIN; footprint Connector_PinHeader_2.54mm:PinHeader_1x01_P2.54mm_Vertical -> Connector_Wire:SolderWire-2sqmm_1x02_P7.8mm_D2mm_OD3.9mm
- J2: value GND -> VOLTMETER; footprint MountingHole:MountingHole_3.2mm_M3_Pad_Via -> Connector_Wire:SolderWire-2sqmm_1x02_P7.8mm_D2mm_OD3.9mm
- J3: value VDD_OUT -> STS3032; footprint MountingHole:MountingHole_3.2mm_M3_Pad_Via -> Connector_JST:JST_XH_B3B-XH-A_1x03_P2.50mm_Vertical
- J4: value GND -> STS3032; footprint MountingHole:MountingHole_3.2mm_M3_Pad_Via -> Connector_JST:JST_XH_B3B-XH-A_1x03_P2.50mm_Vertical
- J5: value SW_VI -> STS3032; footprint Connector_PinHeader_2.54mm:PinHeader_1x01_P2.54mm_Vertical -> Connector_JST:JST_XH_B3B-XH-A_1x03_P2.50mm_Vertical
- J6: value SW_VO -> STS3032; footprint Connector_PinHeader_2.54mm:PinHeader_1x01_P2.54mm_Vertical -> Connector_JST:JST_XH_B3B-XH-A_1x03_P2.50mm_Vertical
- J7: value Conn_01x04 -> 5V ToBottom; footprint Connector_JST:JST_XH_B4B-XH-A_1x04_P2.50mm_Vertical -> Connector_Wire:SolderWire-2sqmm_1x02_P7.8mm_D2mm_OD3.9mm
- J8: value VOLTMETER_V -> 3V3 ToBottom; footprint Connector_PinHeader_2.54mm:PinHeader_1x01_P2.54mm_Vertical -> Connector_Wire:SolderWire-2sqmm_1x02_P7.8mm_D2mm_OD3.9mm
- J9: value VOLTMETER_G -> Bottom_XH; footprint Connector_PinHeader_2.54mm:PinHeader_1x01_P2.54mm_Vertical -> Connector_JST:JST_XH_B2B-XH-A_1x02_P2.50mm_Vertical
- moved J2 182.3 mm to (30.4, 24.3)
- moved J1 173.1 mm to (30.4, 18.3)
- moved J4 156.4 mm to (240.1, 39.4)
- moved J7 107.7 mm to (30.4, 30.2)
- moved J8 62.2 mm to (30.4, 36.2)
- moved J3 62.0 mm to (156.2, 59.7), turned to 90 degrees
- moved J10 25.4 mm to (93.9, 74.3)
- moved J5 20.0 mm to (69.0, 44.5)
- moved J6 19.6 mm to (69.0, 52.3)
- moved J9 13.4 mm to (82.5, 50.9)
Connections:
- J10 pad 1: Net-(J10-Pin_1) -> +5V
- J2 pad 1: GND -> VDD
- J3 pad 1: Net-(J10-Pin_1) -> Motor_SIG
- J4 pad 1: GND -> Motor_SIG
- J5 pad 1: Net-(J5-Pin_1) -> Motor_SIG
- J6 pad 1: Net-(J10-Pin_1) -> Motor_SIG
- J7 pad 1: Net-(J7-Pin_1) -> +5V
- J7 pad 2: Net-(J7-Pin_2) -> GND
- J8 pad 1: Net-(J10-Pin_1) -> +3V3
- J9 pad 1: GND -> Net-(J9-Pin_1)
Other:
- board outline added: 100 x 75 mm

Commit message: パワー
Parts:
- removed J8: 3V3 ToBottom, Connector_Wire:SolderWire-2sqmm_1x02_P7.8mm_D2mm_OD3.9mm
- added C5: 1u, Capacitor_SMD:C_0805_2012Metric, F.Cu at (239.9, 28.3)
- added C6: 1u, Capacitor_SMD:C_0805_2012Metric, F.Cu at (246.3, 29.2)
- added F1: Fuse, Akiduki:FUSE_3557-15, F.Cu at (196.8, 84.5)
- added G***: LOGO, logo:tuton_logo, F.Cu at (226.1, 111.1)
- added J11: Conn_01x04, Connector_JST:JST_XH_B4B-XH-A_1x04_P2.50mm_Vertical, F.Cu at (198.1, 39.4)
- added REF**: MountingHole_3.2mm_M3, MountingHole:MountingHole_3.2mm_M3, F.Cu at (276.3, 78.7)
- added REF**: MountingHole_3.2mm_M3, MountingHole:MountingHole_3.2mm_M3, F.Cu at (241.4, 143.6)
- added REF**: MountingHole_3.2mm_M3, MountingHole:MountingHole_3.2mm_M3, F.Cu at (211.4, 143.6)
- added REF**: MountingHole_3.2mm_M3, MountingHole:MountingHole_3.2mm_M3, F.Cu at (176.4, 78.7)
- added U5: ~, Akiduki:M51957B, F.Cu at (186.1, 84.5)
- added U6: XC6206P332MR-G, Package_TO_SOT_SMD:SOT-23-3, F.Cu at (243.1, 27.9)
- J2: footprint Connector_Wire:SolderWire-2sqmm_1x02_P7.8mm_D2mm_OD3.9mm -> Connector_Wire:SolderWire-0.5sqmm_1x02_P4.6mm_D0.9mm_OD2.1mm
- J7: value 5V ToBottom -> ToLINE; footprint Connector_Wire:SolderWire-2sqmm_1x02_P7.8mm_D2mm_OD3.9mm -> Connector_JST:JST_XH_B6B-XH-A_1x06_P2.50mm_Vertical
- J9: value Bottom_XH -> 3V3 ToMAIN; footprint Connector_JST:JST_XH_B2B-XH-A_1x02_P2.50mm_Vertical -> Connector_Wire:SolderWire-2sqmm_1x02_P7.8mm_D2mm_OD3.9mm
- moved J2 248.4 mm to (268.0, 96.9), turned to 90 degrees
- moved Q1 222.2 mm to (274.4, 91.4), turned to -90 degrees
- moved R9 204.0 mm to (278.3, 92.5), turned to 90 degrees
- moved J6 199.4 mm to (255.3, 123.2)
- moved J7 189.8 mm to (220.0, 40.0)
- moved J1 187.2 mm to (209.5, 73.0)
- moved C4 177.8 mm to (229.9, 48.3), turned to 180 degrees
- moved C3 176.1 mm to (228.0, 57.7), turned to 90 degrees
- moved C1 169.7 mm to (220.3, 65.4), turned to 180 degrees
- moved U2 166.5 mm to (199.4, 115.6), turned to 180 degrees
- moved R6 166.0 mm to (244.7, 54.8), turned to -90 degrees
- moved R5 165.9 mm to (244.7, 51.4), turned to -90 degrees
- moved C2 163.0 mm to (214.0, 64.8)
- moved J9 159.5 mm to (241.9, 44.6), turned to 90 degrees
- moved U1 155.2 mm to (189.2, 97.8), turned to 0 degrees
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Connections:
- C4 pad 1: +3V3 -> 3V3_LED
- J7 pad 1: +5V -> UART3_TX
- J7 pad 2: GND -> UART3_RX
- J9 pad 1: Net-(J9-Pin_1) -> 3V3_LED
- J9 pad 2: Motor_SIG -> GND
- R8 pad 1: +3V3 -> 3V3_LED
- U4 pad 4: +3V3 -> 3V3_LED
- U4 pad 5: +3V3 -> 3V3_LED
Routing:
- net Motor_SIG: track 0.00 -> 272.7 mm
- net Net-(J3-Pin_2): track 0.00 -> 190.4 mm
- net VDD: track 0.00 -> 117.5 mm
- net GND: track 0.00 -> 116.9 mm, vias 0 -> 55
- net Net-(J5-Pin_2): track 0.00 -> 99.7 mm
- net Battery_obs: track 0.00 -> 74.0 mm, vias 0 -> 2
- net Net-(Q1-S): track 0.00 -> 65.1 mm
- net +5V: track 0.00 -> 62.7 mm
- net UART3_RX: track 0.00 -> 31.4 mm
- net +3V3: track 0.00 -> 28.8 mm, vias 0 -> 1
- net UART3_TX: track 0.00 -> 26.3 mm
- net Net-(U5-IN): track 0.00 -> 21.2 mm
- net Net-(J1-Pin_1): track 0.00 -> 16.6 mm
- net 3V3_LED: track 0.00 -> 15.6 mm
- net Net-(Q1-G): track 0.00 -> 15.3 mm
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- added copper zone on F.Cu, net +5V
- added copper zone on F.Cu, net 3V3_LED
- added copper zone on B.Cu, net GND
- added copper zone on F.Cu, net GND
- added copper zone on B.Cu, net Net-(Q1-S)
- added copper zone on F.Cu, net VDD
Other:
- board size 100 x 75 mm -> 110 x 125 mm

Commit message: pdf
Parts:
- removed the G*** at (226.1, 111.1)
- added G***: LOGO, logo:jlcpcb_logo, F.Cu at (217.4, 134.4)
- added G***: LOGO, logo:st_logo, F.Cu at (239.0, 134.4)
- added G***: LOGO, logo:tuton_logo_small, F.Cu at (229.9, 133.9)
- added G***: LOGO, logo:tuton_logo_big, B.Cu at (226.6, 111.8)
- added G***: LOGO, logo:st_logo_big, B.Cu at (226.6, 135.6)
- added G***: LOGO, logo:jlcpcb_logo_big, B.Cu at (228.6, 91.4)
- moved RV1 2.03 mm to (189.2, 116.3)
- moved RV2 1.52 mm to (199.4, 97.5)
Routing:
- net Net-(U1-Trim): track 8.89 -> 10.9 mm
- net Net-(J5-Pin_2): track 99.7 -> 98.4 mm
- net Net-(U2-Trim): track 8.89 -> 10.2 mm
Other:
- board text added: "05-PWR ver.1"
- board text added: "11.1V ->5V OKL ->3.3V OKL ->7.2V TPS5430"
- board text added: "3V3"
- board text added: "3V3L"
- board text added: "5V"
- board text added: "<-FRONT"
- board text added: "BACK->"
- board text added: "BAT"
- board text added: "D"
- board text added: "EN"
- board text added: "G"
- board text added: "GND"
- board text added: "LINE MCU 3V3 REG"
- board text added: "LINE->MAIN"
- board text added: "Lipo 3S 11.1V"
- board text added: "M51957B"
- board text added: "MAIN->LINE"
- board text added: "MOTOR"
- board text added: "OKL 3.3V"
- board text added: "OKL 5V"
- board text added: "OUT"
- board text added: "Pch MOSFET"
- board text added: "RCJ 2025 tuton"
- board text added: "RX<-"
- board text added: "S"
- board text added: "TX->"
- board text added: "ToLINE"
- board text added: "ToMAIN"
- board text added: "Trim"
- board text added: "V"
- board text added: "VBAT"
- board text added: "VDD"
- board text added: "VIN"
- board text added: "VOLTMETER"
