File: 07-STS3032/07-STS3032.kicad_sch (KiCad schematic)
At the start: 11 parts, among them J1 Motor_R1, J2 Motor_R1, J3 Motor_R1, J4 Motor_R1, Q1 2SA1015, U1 MAX485E

Commit message: pdf
Parts:
- removed J1, J2, J3, J4: Motor_R1, symbol Connector_Generic:Conn_01x03
