File: 01-main/01-main.kicad_sch (KiCad schematic)
At the start: 1 part, among them U1 STM32H723ZETx

Commit message: 祝日は進捗を生む日
Parts:
- added BZ1: Buzzer, symbol Device:Buzzer
- added C1, C11, C12, C13, C14, C16, C2, C20, C21, C3, C4, C5, C6, C7, C8: 100nF, symbol Device:C
- added C10: 4.7uF, symbol Device:C
- added C15, C19, C9: 1uF, symbol Device:C
- added C17, C18: 2.2uF, symbol Device:C
- added C22, C23: 1.5pF, symbol Device:C
- added C24, C25: 33pF, symbol Device:C
- added C26, C27, C33, C35, C37, C39: 0.1u, symbol Device:C
- added C28, C30: 10u, symbol Device:C
- added C29, C31: 22u, symbol Device:C
- added C32, C34, C36, C38: 0.33u, symbol Device:C
- added D1, D2: LED, symbol Device:LED
- added FB1: FerriteBead, symbol Device:FerriteBead
- added J1: USB_C_Receptacle_USB2.0, symbol Connector:USB_C_Receptacle_USB2.0
- added J10: front, symbol Connector_Generic:Conn_01x10
- added J11: ToF_R, symbol Connector_Generic:Conn_01x04
- added J12: ToF_RB, symbol Connector_Generic:Conn_01x04
- added J13: ToF_L, symbol Connector_Generic:Conn_01x04
- added J14: ToF_LB, symbol Connector_Generic:Conn_01x04
- added J15, J16: PWR_board_GND, symbol Connector_Generic:Conn_01x01
- added J17: PWR_board_VIN, symbol Connector_Generic:Conn_01x01
- added J18: PWR_board_VOUT, symbol Connector_Generic:Conn_01x01
- added J19: XT60_LiPo, symbol Connector_Generic:Conn_01x02
- added J2: Motor_RF, symbol Connector_Generic:Conn_01x03
- added J20: UI_conn, symbol Connector_Generic:Conn_01x04
- added J21: LOADCELL_R, symbol Connector_Generic:Conn_01x04
- added J22: LOADCELL_L, symbol Connector_Generic:Conn_01x04
- added J23: Conn_01x08, symbol Connector_Generic:Conn_01x08
- added J3: Motor_RB, symbol Connector_Generic:Conn_01x03
- added J4: Motor_LF, symbol Connector_Generic:Conn_01x03
- added J5: Motor_LB, symbol Connector_Generic:Conn_01x03
- added J6: OpenMV, symbol Connector_Generic:Conn_01x04
- added J7, J9: Conn_01x10, symbol Connector_Generic:Conn_01x10
- added J8: Top, symbol Connector_Generic:Conn_02x03_Counter_Clockwise
- added R1: 10K, symbol Device:R
- added R10, R11, R7, R8: 500, symbol Device:R
- added R12, R13, R6, R9: 330k, symbol Device:R
- added R2, R3: 5.1k, symbol Device:R
- added R4, R5: R, symbol Device:R
- added SW1: SW_RST, symbol Switch:SW_Push
- added SW2: SW_BOOT0, symbol Switch:SW_SPDT
- added U10, U7, U8, U9: REG 6V, Package_TO_SOT_SMD:TO-252-2, symbol Regulator_Linear:LF50_TO252
- added U11, U12: NJU77551F, Package_TO_SOT_SMD:SOT-23-5, symbol Amplifier_Operational:OPA196xDBV
- added U13: ~, symbol S11059:S11059
- added U2: CH340E, Package_SO:MSOP-10_3x3mm_P0.5mm, symbol Interface_USB:CH340E
- added U3: ~, symbol MPU6050:MPU6050
- added U4: REG 3V3, Package_TO_SOT_SMD:TO-252-2, symbol Regulator_Linear:LF33_TO252
- added U5: ~, symbol BNO055:AE-BNO055-BO
- added U6: REG 5V, Package_TO_SOT_SMD:TO-252-2, symbol Regulator_Linear:LF50_TO252
- added Y1: 32.768kHz, symbol Device:Crystal
- added Y2: 24MHz, symbol Device:Crystal
Connections:
- net I2C2_SDA: now reaches U1.10 (PF0)
- net I2C2_SDA: now also J12.4 (Pin_4), J23.1 (Pin_1), U3.4 (SDA)
- net I2C3_SCL: now reaches U1.100 (PA8)
- net I2C3_SCL: now also J10.9 (Pin_9), J13.3 (Pin_3)
- net UART4_RX: now reaches U1.103 (PA11)
- net UART4_RX: now also J8.4 (Pin_4)
- net UART4_TX: now reaches U1.104 (PA12)
- net UART4_TX: now also J8.5 (Pin_5)
- net at U1.106 (VCAP): now also C18.1
- net GND: now reaches U1.107 (VSS), U1.120 (VSS), U1.130 (VSS), U1.16 (VSS), U1.38 (VSS), U1.51 (VSS), U1.61 (VSS), U1.83 (VSS), U1.94 (VSS)
- net GND: now also U1.31 (VSSA), BZ1.2 (+), C1.2, C10.2, C11.2, C12.2, C13.2, C14.2, C15.2, C16.2, C17.2, C18.2, C19.2, C2.2, C20.2, C21.1, C22.2, C23.1, C24.1, C25.2, C26.1, C27.2, C28.2, C29.2, C3.2, C30.2, C31.2, C32.2, C33.2, C34.2, C35.2, C36.2, C37.2, C38.2, C39.2, C4.2, C5.2, C6.2, C7.2, C8.2, C9.2, D2.1 (K), J1.A1 (GND), J1.A12 (GND), J1.B1 (GND), J1.B12 (GND), J10.10 (Pin_10), J10.7 (Pin_7), J11.2 (Pin_2), J12.2 (Pin_2), J13.2 (Pin_2), J14.2 (Pin_2), J15.1 (Pin_1), J16.1 (Pin_1), J19.2 (Pin_2), J2.2 (Pin_2), J21.1 (Pin_1), J22.1 (Pin_1), J23.6 (Pin_6), J3.2 (Pin_2), J4.2 (Pin_2), J5.2 (Pin_2), J6.4 (Pin_4), J8.6 (Pin_6), R13.2, R2.2, R3.2, R4.2, R6.2, SW1.1, SW2.3 (C), U10.2 (GND), U11.2 (V-), U12.2 (V-), U13.4 (GND), U2.3 (GND), U3.2 (GND), U4.2 (GND), U5.2 (GND), U6.2 (GND), U7.2 (GND), U8.2 (GND), U9.2 (GND)
- net +3V3: now reaches U1.108 (VDD)
- net +3V3: now also U1.121 (VDD), U1.131 (VDD), U1.143 (PDR_ON), U1.144 (VDD), U1.17 (VDD), U1.30 (VDD), U1.39 (VDD), U1.52 (VDD), U1.6 (VBAT), U1.62 (VDD), U1.72 (VDD), U1.84 (VDD), U1.95 (VDD33USB), C1.1, C10.1, C11.1, C12.1, C13.1, C14.1, C15.1, C16.1, C2.1, C29.1, C3.1, C4.1, C5.1, C6.1, C7.1, FB1.1, J10.1 (Pin_1), J11.1 (Pin_1), J12.1 (Pin_1), J13.1 (Pin_1), J14.1 (Pin_1), J21.4 (Pin_4), J22.4 (Pin_4), J23.3 (Pin_3), SW2.1 (A), U11.5 (V+), U12.5 (V+), U13.1 (+V), U3.1 (VCC), U4.3 (VO), U5.1 (VIN)
- net I2C2_SCL: now reaches U1.11 (PF1)
- net I2C2_SCL: now also J12.3 (Pin_3), J23.2 (Pin_2), U3.3 (SCL)
- net Buzzer: now reaches U1.110 (PA15(JTDI))
- net Buzzer: now also BZ1.1 (-)
- net UART2_TX: now reaches U1.119 (PD5)
- net UART2_TX: now also J8.2 (Pin_2)
- net UART2_RX: now reaches U1.122 (PD6)
- net UART2_RX: now also J8.3 (Pin_3)
- net line_photo_RR: now reaches U1.13 (PF3)
- net line_photo_RR: now also J9.10 (Pin_10)
- net I2C1_SCL: now reaches U1.136 (PB6)
- net I2C1_SCL: now also J11.3 (Pin_3), J23.8 (Pin_8), U13.3 (SCL), U5.4 (SCL)
- net I2C1_SDA: now reaches U1.137 (PB7)
- net I2C1_SDA: now also J11.4 (Pin_4), J23.7 (Pin_7), U13.2 (SDA), U5.3 (SDA)
- net BOOT0: now reaches U1.138 (BOOT0)
- net BOOT0: now also R1.2
- net front_photo_1: now reaches U1.15 (PF5)
- net front_photo_1: now also J10.2 (Pin_2)
- net LOADCEL_R: now reaches U1.18 (PF6)
- net LOADCEL_R: now also R9.1, U11.1
- net line_photo_front: now reaches U1.19 (PF7)
- net line_photo_front: now also J23.5 (Pin_5)
- net line_photo_center: now reaches U1.21 (PF9)
- net line_photo_center: now also J23.4 (Pin_4)
- net LOADCEL_L: now reaches U1.22 (PF10)
- net LOADCEL_L: now also R12.1, U12.1
- net at U1.23 (PH0): now also C24.2, Y2.2
- net at U1.24 (PH1): now also C25.1, Y2.1
- net NRST: now reaches U1.25 (NRST)
- net NRST: now also C21.2, SW1.2
- net line_photo_R_9: now reaches U1.26 (PC0)
- net line_photo_R_9: now also J9.9 (Pin_9)
- net line_photo_R_8: now reaches U1.27 (PC1)
- net line_photo_R_8: now also J9.8 (Pin_8)
- net line_photo_LL: now reaches U1.29 (PC3_C)
- net line_photo_LL: now also J7.10 (Pin_10)
- net +3.3VA: now reaches U1.32 (VREF+)
- net +3.3VA: now also U1.33 (VDDA), C19.1, C20.1, C8.1, C9.1, FB1.2
- net line_photo_R_7: now reaches U1.34 (PA0)
- net line_photo_R_7: now also J9.7 (Pin_7)
- net line_photo_R_6: now reaches U1.35 (PA1)
- net line_photo_R_6: now also J9.6 (Pin_6)
- net line_photo_R_5: now reaches U1.36 (PA2)
- net line_photo_R_5: now also J9.5 (Pin_5)
- net line_photo_R_4: now reaches U1.37 (PA3)
- net line_photo_R_4: now also J9.4 (Pin_4)
- net line_photo_R_3: now reaches U1.40 (PA4)
- net line_photo_R_3: now also J9.3 (Pin_3)
- net line_photo_R_2: now reaches U1.41 (PA5)
- net line_photo_R_2: now also J9.2 (Pin_2)
- net line_photo_R_1: now reaches U1.42 (PA6)
- net line_photo_R_1: now also J9.1 (Pin_1)
- net line_photo_L_1: now reaches U1.43 (PA7)
- net line_photo_L_1: now also J7.1 (Pin_1)
- net line_photo_L_2: now reaches U1.44 (PC4)
- net line_photo_L_2: now also J7.2 (Pin_2)
- net line_photo_L_3: now reaches U1.45 (PC5)
- net line_photo_L_3: now also J7.3 (Pin_3)
- net line_photo_L_4: now reaches U1.46 (PB0)
- net line_photo_L_4: now also J7.4 (Pin_4)
- net line_photo_L_5: now reaches U1.47 (PB1)
- net line_photo_L_5: now also J7.5 (Pin_5)
- net line_photo_L_6: now reaches U1.49 (PF11)
- net line_photo_L_6: now also J7.6 (Pin_6)
- net line_photo_L_7: now reaches U1.50 (PF12)
- net line_photo_L_7: now also J7.7 (Pin_7)
- net line_photo_L_8: now reaches U1.53 (PF13)
- net line_photo_L_8: now also J7.8 (Pin_8)
- net line_photo_L_9: now reaches U1.54 (PF14)
- net line_photo_L_9: now also J7.9 (Pin_9)
- net MotorRF: now reaches U1.60 (PE9)
- net MotorRF: now also J2.3 (Pin_3)
- net MotorRB: now reaches U1.64 (PE11)
- net MotorRB: now also J3.3 (Pin_3)
- net MotorLF: now reaches U1.66 (PE13)
- net MotorLF: now also J4.3 (Pin_3)
- net MotorLB: now reaches U1.67 (PE14)
- net MotorLB: now also J5.3 (Pin_3)
- net UART3_TX: now reaches U1.69 (PB10)
- net UART3_TX: now also J6.2 (Pin_2)
- net UART3_RX: now reaches U1.70 (PB11)
- net UART3_RX: now also J6.3 (Pin_3)
- net at U1.71 (VCAP): now also C17.1
- net UART1_TX: now reaches U1.75 (PB14)
- net UART1_TX: now also U2.9 (RXD)
- net UART1_RX: now reaches U1.76 (PB15)
- net UART1_RX: now also U2.8 (TXD)
- net PC14: now reaches U1.8 (PC14)
- net PC14: now also C22.1, Y1.2
- net I2C4_SCL: now reaches U1.81 (PD12)
- net I2C4_SCL: now also J14.3 (Pin_3)
- net I2C4_SDA: now reaches U1.82 (PD13)
- net I2C4_SDA: now also J14.4 (Pin_4)
- net UI_toggle: now reaches U1.88 (PG3)
- net UI_toggle: now also J20.1 (Pin_1)
- net UI_push1: now reaches U1.89 (PG4)
- net UI_push1: now also J20.2 (Pin_2)
- net PC15: now reaches U1.9 (PC15)
- net PC15: now also C23.2, Y1.1
- net UI_push2: now reaches U1.90 (PG5)
- net UI_push2: now also J20.3 (Pin_3)
- net UI_push3: now reaches U1.91 (PG6)
- net UI_push3: now also J20.4 (Pin_4)
- net I2C3_SDA: now reaches U1.99 (PC9)
- net I2C3_SDA: now also J10.8 (Pin_8), J13.4 (Pin_4)
- new net: C33.1, J2.1 (Pin_1), U7.3 (VO)
- new net: C35.1, J3.1 (Pin_1), U8.3 (VO)
- new net: J17.1 (Pin_1), J19.1 (Pin_1)
- new net: J22.2 (Pin_2), R10.1
- new net: J22.3 (Pin_3), R11.2
- new net: R10.2, R13.1, U12.3 (+)
- new net: J1.A5 (CC1), R3.1
- new net: J21.2 (Pin_2), R7.1
- new net: J21.3 (Pin_3), R8.2
- new net: R11.1, R12.2, U12.4 (-)
- new net: R6.1, R7.2, U11.3 (+)
- new net: R8.1, R9.2, U11.4 (-)
- new net: C37.1, J4.1 (Pin_1), U9.3 (VO)
- new net: J1.B5 (CC2), R2.1
- new net: R1.1, SW2.2 (B)
- new net: D2.2 (A), R5.2
- new net: D1.1 (K), R4.1
- new net: C26.2, U2.10 (V3)
- new net: D1.2 (A), J1.A4 (VBUS), J1.A9 (VBUS), J1.B4 (VBUS), J1.B9 (VBUS)
- new net: C39.1, J5.1 (Pin_1), U10.3 (VO)
- new net: R5.1, U2.6 (TNOW)
- new net +5V: C27.1, C31.1, J6.1 (Pin_1), U2.7 (VCC), U6.3 (VO)
- new net D+: J1.A6 (D+), J1.B6 (D+), U2.1 (UD+)
- new net D-: J1.A7 (D-), J1.B7 (D-), U2.2 (UD-)
- new net VDD: C28.1, C30.1, C32.1, C34.1, C36.1, C38.1, J18.1 (Pin_1), J8.1 (Pin_1), U10.1 (VI), U4.1 (VI), U6.1 (VI), U7.1 (VI), U8.1 (VI), U9.1 (VI)
- no-connect marks 0 -> 77
Other:
- note added: "CONN"
- note added: "LINE_SENSOR"
- note added: "LOADCELL"
- note added: "MOTOR"
- note added: "POWER"
- note added: "SENSOR"
- note added: "STM32H723ZGT6"
- moved on the sheet: U1

Commit message: 全国行きたかった
Parts:
- R10, R11, R7, R8: value 500 -> 330
Connections:
- net GND: now also J10.3 (Pin_3), J10.4 (Pin_4), J10.5 (Pin_5), J10.6 (Pin_6)
- no-connect marks 77 -> 73
Other:
- note added: "LINE SENSOR"
- note removed: "LINE_SENSOR"

Commit message: がんばる
Parts:
- removed C10: 4.7uF, symbol Device:C
- removed C11, C12, C13, C14, C16, C20, C21, C4, C5, C6, C7, C8: 100nF, symbol Device:C
- removed C15, C19, C9: 1uF, symbol Device:C
- removed C17, C18: 2.2uF, symbol Device:C
- removed C22, C23: 1.5pF, symbol Device:C
- removed C24, C25: 33pF, symbol Device:C
- removed C26, C27, C33, C35, C37, C39: 0.1u, symbol Device:C
- removed C28, C30: 10u, symbol Device:C
- removed C29, C31: 22u, symbol Device:C
- removed C32, C34, C36, C38: 0.33u, symbol Device:C
- removed D1, D2: LED, symbol Device:LED
- removed FB1: FerriteBead, symbol Device:FerriteBead
- removed J1: USB_C_Receptacle_USB2.0, symbol Connector:USB_C_Receptacle_USB2.0
- removed J10: front, symbol Connector_Generic:Conn_01x10
- removed J11: ToF_R, symbol Connector_Generic:Conn_01x04
- removed J12: ToF_RB, symbol Connector_Generic:Conn_01x04
- removed J13: ToF_L, symbol Connector_Generic:Conn_01x04
- removed J14: ToF_LB, symbol Connector_Generic:Conn_01x04
- removed J15, J16: PWR_board_GND, symbol Connector_Generic:Conn_01x01
- removed J17: PWR_board_VIN, symbol Connector_Generic:Conn_01x01
- removed J18: PWR_board_VOUT, symbol Connector_Generic:Conn_01x01
- removed J19: XT60_LiPo, symbol Connector_Generic:Conn_01x02
- removed J2: Motor_RF, symbol Connector_Generic:Conn_01x03
- removed J20: UI_conn, symbol Connector_Generic:Conn_01x04
- removed J21: LOADCELL_R, symbol Connector_Generic:Conn_01x04
- removed J22: LOADCELL_L, symbol Connector_Generic:Conn_01x04
- removed J23: Conn_01x08, symbol Connector_Generic:Conn_01x08
- removed J3: Motor_RB, symbol Connector_Generic:Conn_01x03
- removed J6: OpenMV, symbol Connector_Generic:Conn_01x04
- removed J7, J9: Conn_01x10, symbol Connector_Generic:Conn_01x10
- removed J8: Top, symbol Connector_Generic:Conn_02x03_Counter_Clockwise
- removed R6: 330k, symbol Device:R
- removed R7, R8: 330, symbol Device:R
- removed SW1: SW_RST, symbol Switch:SW_Push
- removed SW2: SW_BOOT0, symbol Switch:SW_SPDT
- removed U1: STM32H723ZETx, Package_QFP:LQFP-144_20x20mm_P0.5mm, symbol MCU_ST_STM32H7:STM32H723ZETx
- removed U10, U7, U8, U9: REG 6V, Package_TO_SOT_SMD:TO-252-2, symbol Regulator_Linear:LF50_TO252
- removed U11, U12: NJU77551F, Package_TO_SOT_SMD:SOT-23-5, symbol Amplifier_Operational:OPA196xDBV
- removed U13: ~, symbol S11059:S11059
- removed U2: CH340E, Package_SO:MSOP-10_3x3mm_P0.5mm, symbol Interface_USB:CH340E
- removed U3: ~, symbol MPU6050:MPU6050
- removed U4: REG 3V3, Package_TO_SOT_SMD:TO-252-2, symbol Regulator_Linear:LF33_TO252
- removed U5: ~, symbol BNO055:AE-BNO055-BO
- removed U6: REG 5V, Package_TO_SOT_SMD:TO-252-2, symbol Regulator_Linear:LF50_TO252
- removed Y1: 32.768kHz, symbol Device:Crystal
- removed Y2: 24MHz, symbol Device:Crystal
- added J2: WRITER CONN, Connector_PinHeader_2.54mm:PinHeader_2x04_P2.54mm_Vertical, symbol Connector_Generic:Conn_02x04_Counter_Clockwise
- added J2: LOADCELL_R, symbol Connector_Generic:Conn_01x04
- added J3: LOADCELL_L, symbol Connector_Generic:Conn_01x04
- added J6, J7: Motor_R1, symbol Connector_Generic:Conn_01x03
- added J8: ToLINE, symbol Connector_Generic:Conn_01x04
- added Q1: 2SA1015, Package_TO_SOT_THT:TO-92_Inline, symbol Transistor_BJT:2SA1015
- added R14, R15, R16: 330k, symbol Device:R
- added U2: STM32F446RETx, Package_QFP:LQFP-64_10x10mm_P0.5mm, symbol MCU_ST_STM32F4:STM32F446RETx
- added U2: MAX485E, symbol Interface_UART:MAX485E
- added U3: ~, symbol BNO055:AE-BNO055-BO
- added U5, U6: NJU77551F, Package_TO_SOT_SMD:SOT-23-5, symbol Amplifier_Operational:OPA196xDBV
- C1: value 100nF -> 0.1u
- C2: value 100nF -> 100n
- C3: value 100nF -> 4.7u
- J4: value Motor_LF -> Motor_R1
- J5: value Motor_LB -> Motor_R1
- R1: value 10K -> 220
- R12, R9: value 330k -> 330
- R2: value 5.1k -> 7.5k
- R3: value 5.1k -> 2.2k
- R4: value R -> 2.2k
- R5: value R -> 10k; footprint (none) -> Resistor_SMD:R_0805_2012Metric; LCSC (none) -> C17414
Connections:
- net MotorLB is gone; now on net GND: J5.3 (Pin_3)
- net MotorLF is gone; now on net GND: J4.3 (Pin_3)
- net +3V3: now also J2.4 (Pin_4), J2.8 (Pin_8), J3.4 (Pin_4), U2.1 (VBAT), U2.13 (VDDA), U2.19 (VDD), U2.32 (VDD), U2.48 (VDD), U2.64 (VDD), U3.1 (VIN), U5.5 (V+), U6.5 (V+); no longer C1.1, C2.1, C3.1
- net +5V: now also C1.1, R3.1, Q1.2 (C), U2.8 (VCC)
- net BOOT0: now also R5.1, J2.5 (Pin_5), U2.60 (BOOT0); no longer R1.2
- net GND: now also C2.1, R1.2, R4.1, R5.2, J2.1 (Pin_1), J2.6 (Pin_6), J3.1 (Pin_1), J6.3 (Pin_3), J7.3 (Pin_3), R15.2, U2.12 (VSSA), U2.18 (VSS), U2.31 (VSS), U2.47 (VSS), U2.5 (GND), U2.63 (VSS), U3.2 (GND), U5.2 (V-), U6.2 (V-); no longer C2.2, J4.2 (Pin_2), J5.2 (Pin_2), R2.2, R3.2, R4.2
- net I2C1_SCL: now also U2.58 (PB6), U3.4 (SCL)
- net I2C1_SDA: now also U2.59 (PB7), U3.3 (SDA)
- net I2C2_SCL: now also U2.29 (PB10)
- net I2C2_SDA: now also U2.53 (PC12)
- net LOADCEL_L: now also R16.1, U6.1; no longer R12.1
- net LOADCEL_R: now also R14.1, U5.1; no longer R9.1
- net NRST: now also C2.2, J2.3 (Pin_3), U2.7 (NRST)
- net UART1_RX: now also J2.2 (Pin_2), U2.43 (PA10)
- net UART1_TX: now also J2.4 (Pin_4), U2.42 (PA9)
- net at R10.1: now also R14.2, U5.4 (-)
- net at R11.2: now also R15.1, U6.3 (+)
- net at R13.1: now also R9.2, U5.3 (+); no longer R10.2
- net at R11.1: now also J3.2 (Pin_2); no longer R12.2
- net STS_SIG: now reaches J4.1 (Pin_1)
- net STS_SIG: now also J5.1 (Pin_1), J6.1 (Pin_1), J7.1 (Pin_1), U2.6 (A)
- net at R2.1: now also Q1.3 (B)
- net at R1.1: now also Q1.1 (E), U2.2 (~{RE}), U2.3 (DE)
- net Buzzer: no longer names the net of BZ1.1 (-)
- new net: J3.3 (Pin_3), R12.2
- new net: R12.1, R16.2, U6.4 (-)
- new net: J2.2 (Pin_2), R9.1
- new net: J2.3 (Pin_3), R10.2
- new net: C3.1, U2.30 (VCAP_1)
- new net: R3.2, R4.2, U2.7 (B)
- new net: R2.2, U2.4 (DI)
- new net +6V: J4.2 (Pin_2), J5.2 (Pin_2), J6.2 (Pin_2), J7.2 (Pin_2)
- no-connect marks 73 -> 6
Other:
- note removed: "CONN"
- note removed: "LINE SENSOR"
- note removed: "LOADCELL"
- note removed: "MOTOR"
- note removed: "POWER"
- note removed: "SENSOR"
- note removed: "STM32H723ZGT6"

Commit message: いっぱい増えた
Parts:
- removed U2: STM32F446RETx, Package_QFP:LQFP-64_10x10mm_P0.5mm, symbol MCU_ST_STM32F4:STM32F446RETx
- added C1: 10u, Capacitor_SMD:C_0603_1608Metric, symbol Device:C
- added C10, C12, C13, C5, C7, C8, C9: 100n, Capacitor_SMD:C_0402_1005Metric, symbol Device:C
- added C11, C6: 4.7u, Capacitor_SMD:C_0402_1005Metric, symbol Device:C
- added C14: 1u, Capacitor_SMD:C_0402_1005Metric, symbol Device:C
- added C4: 100u, Capacitor_SMD:C_1206_3216Metric, symbol Device:C
- added FB1: FerriteBead, Resistor_SMD:R_0805_2012Metric, symbol Device:FerriteBead
- added J1: ToTOP, symbol Connector_Generic:Conn_01x04
- added J11: ToFRONT, symbol Connector_Generic:Conn_01x04
- added J2: ST-LINK, Connector_PinHeader_2.54mm:PinHeader_1x04_P2.54mm_Vertical, symbol Connector_Generic:Conn_01x04
- added R2: 10k, Resistor_SMD:R_0603_1608Metric, symbol Device:R
- added U1: ~, Package_TO_SOT_SMD:SOT-223-6, symbol JLCPCB_items:TPS7A4533DCQR
- added U2: ~, Package_TO_SOT_SMD:TO-252-3_TabPin2, symbol JLCPCB_items:BA50BC0FP
- added U3: STM32F446RETx, Package_QFP:LQFP-64_10x10mm_P0.5mm, symbol MCU_ST_STM32F4:STM32F446RETx
- C2: value 100n -> 10u; footprint (none) -> Capacitor_SMD:C_0603_1608Metric; LCSC (none) -> C3015157
- C3: value 4.7u -> 0.33u; footprint (none) -> Capacitor_SMD:C_0805_2012Metric; LCSC (none) -> C2961026
- R5: footprint Resistor_SMD:R_0805_2012Metric -> Resistor_SMD:R_0603_1608Metric; LCSC C17414 -> C137819
Connections:
- net +3V3: now also C2.1, C10.2, C11.1, C12.2, C7.2, C8.2, C9.2, FB1.1, U1.4 (OUT), U1.5 (SENSE), U3.1 (VBAT), U3.19 (VDD), U3.32 (VDD), U3.48 (VDD), U3.64 (VDD)
- net +5V: now also C4.1, U2.3 (OUT)
- net BOOT0: now also U3.60 (BOOT0)
- net GND: now also C2.2, C1.2, C10.1, C11.2, C12.1, C13.1, C14.1, C4.2, C5.1, C6.2, C7.1, C8.1, C9.1, J2.4 (Pin_4), R2.2, U1.3 (GND), U1.6 (GND), U2.2 (GND), U3.12 (VSSA), U3.18 (VSS), U3.31 (VSS), U3.47 (VSS), U3.63 (VSS); no longer C2.1
- net I2C1_SCL: now also U3.58 (PB6)
- net I2C1_SDA: now also U3.59 (PB7)
- net I2C2_SCL: now also U3.29 (PB10)
- net I2C2_SDA: now also U3.53 (PC12)
- net NRST: now also C5.2, J2.3 (Pin_3), U3.7 (NRST); no longer C2.2
- net UART1_RX: now also U3.43 (PA10)
- net UART1_TX: now also U3.42 (PA9)
- net VDD: now reaches C3.1
- net VDD: now also C1.1, U1.1 (SHDN), U1.2 (IN), U2.1 (IN)
- new net: C13.2, C14.2, FB1.2, U3.13 (VDDA)
- new net: R2.1, U3.28 (PB2)
- new net: C6.1, U3.30 (VCAP_1)
- new net SWCLK: J2.1 (Pin_1), U3.49 (PA14)
- new net SWDIO: J2.2 (Pin_2), U3.46 (PA13)
- new net UART2_RX: U3.17 (PA3)
- new net UART2_TX: U3.16 (PA2)
- new net UART3_RX: U3.25 (PC5)
- new net UART3_TX: U3.51 (PC10)
- new net UART4_RX: U3.15 (PA1)
- new net UART4_TX: U3.14 (PA0)
Other:
- moved on the sheet: BZ1, C1, J8, Q1, R1, R2, R3, R4, U2, U3

Commit message: わああ
Parts:
- removed C3: 0.33u, Capacitor_SMD:C_0805_2012Metric, symbol Device:C
- removed C4: 100u, Capacitor_SMD:C_1206_3216Metric, symbol Device:C
- removed J1: ToTOP, symbol Connector_Generic:Conn_01x04
- removed J11: ToFRONT, symbol Connector_Generic:Conn_01x04
- removed J2: WRITER CONN, Connector_PinHeader_2.54mm:PinHeader_2x04_P2.54mm_Vertical, symbol Connector_Generic:Conn_02x04_Counter_Clockwise
- removed J4, J5, J6, J7: Motor_R1, symbol Connector_Generic:Conn_01x03
- removed U1: ~, Package_TO_SOT_SMD:SOT-223-6, symbol JLCPCB_items:TPS7A4533DCQR
- removed U2: ~, Package_TO_SOT_SMD:TO-252-3_TabPin2, symbol JLCPCB_items:BA50BC0FP
- removed U5, U6: NJU77551F, Package_TO_SOT_SMD:SOT-23-5, symbol Amplifier_Operational:OPA196xDBV
- added D1: LED_GREEN, LED_SMD:LED_1206_3216Metric, symbol Device:LED
- added D2: LED_ORANGE, LED_SMD:LED_1206_3216Metric, symbol Device:LED
- added J1: USB_C_Receptacle_USB2.0, Connector_USB:USB_C_Receptacle_GCT_USB4105-xx-A_16P_TopMnt_Horizontal, symbol Connector:USB_C_Receptacle_USB2.0
- added J10: arm2, Connector_PinHeader_2.54mm:PinHeader_1x03_P2.54mm_Vertical, symbol Connector_Generic:Conn_01x03
- added J11: handL, Connector_PinHeader_2.54mm:PinHeader_1x03_P2.54mm_Vertical, symbol Connector_Generic:Conn_01x03
- added J12: handR, Connector_PinHeader_2.54mm:PinHeader_1x03_P2.54mm_Vertical, symbol Connector_Generic:Conn_01x03
- added J13: back, Connector_PinHeader_2.54mm:PinHeader_1x03_P2.54mm_Vertical, symbol Connector_Generic:Conn_01x03
- added J15, J16, J17: YOBI, Connector_PinSocket_2.54mm:PinSocket_1x04_P2.54mm_Vertical, symbol Connector_Generic:Conn_01x04
- added J18, J19, J20: PWR, Connector_PinSocket_2.54mm:PinSocket_1x04_P2.54mm_Vertical, symbol Connector_Generic:Conn_01x04
- added J21: I2C, Connector_PinSocket_2.54mm:PinSocket_1x04_P2.54mm_Vertical, symbol Connector_Generic:Conn_01x04
- added J3: ToFront, Connector_JST:JST_XH_B4B-XH-A_1x04_P2.50mm_Vertical, symbol Connector_Generic:Conn_01x04
- added J4: 5V IN, Connector_AMASS:AMASS_XT60PW-M_1x02_P7.20mm_Horizontal, symbol Connector_Generic:Conn_01x02
- added J5: 3V3 IN, Connector_AMASS:AMASS_XT60PW-M_1x02_P7.20mm_Horizontal, symbol Connector_Generic:Conn_01x02
- added J9: arm1, Connector_PinHeader_2.54mm:PinHeader_1x03_P2.54mm_Vertical, symbol Connector_Generic:Conn_01x03
- added R1, R2: 5.1k, Resistor_SMD:R_0805_2012Metric, symbol Device:R
- added R15, R16, R17, R18: 10k, Resistor_SMD:R_0603_1608Metric, symbol Device:R
- added R3, R4: 75, Resistor_SMD:R_0805_2012Metric, symbol Device:R
- added SW1: NRST, Button_Switch_THT:SW_PUSH_6mm, symbol Switch:SW_Push
- added SW2: BOOT0, Button_Switch_THT:SW_PUSH_6mm, symbol Switch:SW_Push
- added U1: CH340E, Package_SO:MSOP-10_3x3mm_P0.5mm, symbol Interface_USB:CH340E
- added U13: ~, Akiduki:MPU6050, symbol MPU6050:MPU6050
- added U14: LM358, Package_SO:SOIC-8_3.9x4.9mm_P1.27mm, symbol Amplifier_Operational:LM358
- added U2, U4, U5, U7: ~, tuton:vl53l0x_vertical, symbol tuton_module:vl53l0x_module
- added U6: ~, XIAO:XIAO_Board, symbol XIAO:XIAO_ESP32C3
- BZ1: footprint (none) -> Buzzer_Beeper:Buzzer_TDK_PS1240P02BT_D12.2mm_H6.5mm
- C1: value 0.1u -> 100n; footprint (none) -> Capacitor_SMD:C_0402_1005Metric; LCSC (none) -> C1525
- C1, C2: value 10u -> 100n; footprint Capacitor_SMD:C_0603_1608Metric -> Capacitor_SMD:C_0402_1005Metric; LCSC C3015157 -> C1525
- C10, C12, C13, C5, C7, C8, C9: LCSC C3012377 -> C1525
- C11, C6: LCSC C7472956 -> C23733
- C14: LCSC C3012378 -> C52923
- J1: renamed from J8; footprint (none) -> Connector_JST:JST_XH_S4B-XH-A_1x04_P2.50mm_Horizontal
- J2: value ST-LINK -> ToTop; footprint Connector_PinHeader_2.54mm:PinHeader_1x04_P2.54mm_Vertical -> Connector_JST:JST_XH_B4B-XH-A_1x04_P2.50mm_Vertical
- J7: renamed from J2; footprint (none) -> Connector_JST:JST_XH_B4B-XH-A_1x04_P2.50mm_Vertical
- J8: renamed from J3; footprint (none) -> Connector_JST:JST_XH_B4B-XH-A_1x04_P2.50mm_Vertical
- R1: value 220 -> 20k; footprint (none) -> Resistor_SMD:R_0603_1608Metric; LCSC (none) -> C4184
- R10: renamed from R14; footprint (none) -> Resistor_SMD:R_0603_1608Metric; LCSC (none) -> C23137
- R11: renamed from R15; footprint (none) -> Resistor_SMD:R_0603_1608Metric; LCSC (none) -> C23137
- R12: renamed from R16; footprint (none) -> Resistor_SMD:R_0603_1608Metric; LCSC (none) -> C23137
- R2: footprint (none) -> Resistor_SMD:R_0603_1608Metric; LCSC (none) -> C23234
- R3, R4: footprint (none) -> Resistor_SMD:R_0603_1608Metric; LCSC (none) -> C4190
- R4: renamed from R9; footprint (none) -> Resistor_SMD:R_0603_1608Metric; LCSC (none) -> C23138
- R5: renamed from R10; footprint (none) -> Resistor_SMD:R_0603_1608Metric; LCSC (none) -> C23138
- R6: renamed from R11; footprint (none) -> Resistor_SMD:R_0603_1608Metric; LCSC (none) -> C23138
- R7: renamed from R12; footprint (none) -> Resistor_SMD:R_0603_1608Metric; LCSC (none) -> C23138
- R9: renamed from R13; footprint (none) -> Resistor_SMD:R_0603_1608Metric; LCSC (none) -> C23137
- U1: renamed from U3; footprint (none) -> Akiduki:BNO055
- U2: value MAX485E -> MAX485ESA; footprint (none) -> Package_SO:SOP-8_3.9x4.9mm_P1.27mm; LCSC (none) -> C668206
Connections:
- net VDD is gone; now on net +5V: C1.1
- net +3V3: now also J19.1 (Pin_1), J19.2 (Pin_2), J19.3 (Pin_3), J19.4 (Pin_4), J3.1 (Pin_1), J5.1 (Pin_1), R15.2, R16.1, R17.2, R18.1, SW2.1, U13.1 (VCC), U14.8 (V+), U2.1 (3V3), U4.1 (3V3), U5.1 (3V3), U7.1 (3V3); no longer C2.1
- net +5V: now also J2.1 (Pin_1), J10.2 (Pin_2), J11.2 (Pin_2), J12.2 (Pin_2), J13.2 (Pin_2), J18.1 (Pin_1), J18.2 (Pin_2), J18.3 (Pin_3), J18.4 (Pin_4), J4.1 (Pin_1), J9.2 (Pin_2), U1.7 (VCC), U6.14 (5V)
- net BOOT0: now also SW2.2
- net GND: now also C2.1, J1.A1 (GND), J1.A12 (GND), J1.B1 (GND), J1.B12 (GND), J10.3 (Pin_3), J11.3 (Pin_3), J12.3 (Pin_3), J13.3 (Pin_3), J20.1 (Pin_1), J20.2 (Pin_2), J20.3 (Pin_3), J20.4 (Pin_4), J3.4 (Pin_4), J4.2 (Pin_2), J5.2 (Pin_2), J9.3 (Pin_3), R1.1, R2.1, R3.2, R4.2, SW1.1, U1.3 (GND), U13.2 (GND), U14.4 (V-), U2.2 (GND), U4.2 (GND), U5.2 (GND), U6.13 (GND), U7.2 (GND); no longer C2.2
- net I2C1_SCL: now also J21.1 (Pin_1), R15.1, U2.3 (SCL), U4.3 (SCL), U5.3 (SCL), U7.3 (SCL)
- net I2C1_SDA: now also J21.2 (Pin_2), R16.2, U2.4 (SDA), U4.4 (SDA), U5.4 (SDA), U7.4 (SDA)
- net I2C2_SCL: now also J21.3 (Pin_3), R17.1, U13.3 (SCL)
- net I2C2_SDA: now also U3.55 (PB3), J21.4 (Pin_4), R18.2, U13.4 (SDA); no longer U3.53 (PC12)
- net LOADCEL_L: now also U3.9 (PC1), U14.1
- net LOADCEL_R: now also U3.8 (PC0), U14.7
- net NRST: now also SW1.2; no longer J2.3 (Pin_3)
- net STS_SIG: now also J1.3 (Pin_3)
- net UART1_RX: now also U1.8 (TXD)
- net UART1_TX: now also U1.9 (RXD)
- net UART2_RX: now also J1.1 (Pin_1)
- net UART2_TX: now also J1.2 (Pin_2)
- net UART3_RX: now also U2.1 (RO)
- net UART3_TX: now also R2.2, U2.4 (DI)
- net UART4_RX: now also J3.2 (Pin_2)
- net UART4_TX: now also J3.3 (Pin_3)
- net buzzer: now reaches BZ1.1 (-)
- net buzzer: now also U3.27 (PB1)
- net at R11.1, R6.2: now also U14.3 (+)
- net at R12.2, R7.1: now also U14.2 (-)
- net at R4.2, R9.1: now also U14.5 (+)
- net at R10.2, R5.1: now also U14.6 (-)
- net at U3.11 (PC3): now also J17.4 (Pin_4)
- net at U3.2 (PC13): now also J16.3 (Pin_3)
- net servo3: now reaches U3.21 (PA5)
- net servo3: now also J11.1 (Pin_1)
- net servo4: now reaches U3.22 (PA6)
- net servo4: now also J12.1 (Pin_1)
- net servo5: now reaches U3.23 (PA7)
- net servo5: now also J13.1 (Pin_1)
- net at U3.24 (PC4): now also J17.3 (Pin_3)
- net servo6: now reaches U3.26 (PB0)
- net at U3.3 (PC14): now also J16.2 (Pin_2)
- net at U3.34 (PB13): now also J15.2 (Pin_2)
- net at U3.35 (PB14): now also J15.3 (Pin_3)
- net at U3.36 (PB15): now also J15.4 (Pin_4)
- net UART6_TX: now reaches U3.37 (PC6)
- net UART6_TX: now also U6.8 (D7)
- net UART6_RX: now reaches U3.38 (PC7)
- net UART6_RX: now also U6.7 (D6)
- net at U3.39 (PC8): now also J17.2 (Pin_2)
- net at U3.4 (PC15): now also J16.1 (Pin_1)
- net at U3.40 (PC9): now also J17.1 (Pin_1)
- net servo1: now reaches U3.41 (PA8)
- net servo1: now also J9.1 (Pin_1)
- net servo2: now reaches U3.44 (PA11)
- net servo2: now also J10.1 (Pin_1)
- net XSHUT1: now reaches U3.45 (PA12)
- net XSHUT1: now also U2.5 (XSHUT)
- net XSHUT4: now reaches U3.50 (PA15)
- net XSHUT4: now also U7.5 (XSHUT)
- net at U3.52 (PC11): now also J16.4 (Pin_4)
- net UART5_RX: now reaches U3.54 (PD2)
- net UART5_RX: now also J2.2 (Pin_2)
- net at U3.57 (PB5): now also J15.1 (Pin_1)
- net BAT: now reaches U3.62 (PB9)
- net BAT: now also J1.4 (Pin_4)
- net SWCLK renamed XSHUT3
- net XSHUT3: now also U5.5 (XSHUT); no longer J2.1 (Pin_1)
- net SWDIO renamed XSHUT2
- net XSHUT2: now also U4.5 (XSHUT); no longer J2.2 (Pin_2)
- new net: C2.2, U1.10 (V3)
- new net: J1.B5 (CC2), R2.2
- new net: D1.2 (A), J1.A4 (VBUS), J1.A9 (VBUS), J1.B4 (VBUS), J1.B9 (VBUS)
- new net: J1.A5 (CC1), R1.2
- new net: D2.2 (A), U1.6 (TNOW)
- new net: D1.1 (K), R3.1
- new net: D2.1 (K), R4.1
- new net D+: J1.A6 (D+), J1.B6 (D+), U1.1 (UD+)
- new net D-: J1.A7 (D-), J1.B7 (D-), U1.2 (UD-)
- new net UART5_TX: J2.3 (Pin_3), U3.53 (PC12)
- no-connect marks 6 -> 34
Other:
- note added: "CONN"
- note added: "Debugger"
- note added: "GYRO"
- note added: "I2C Pullup"
- note added: "LOADCELL"
- note added: "MAIN F446"
- note added: "RS485"
- note added: "SERVO"
- note added: "ToF"
- note added: "UART1:WRITER UART2:LINE UART3:STS3032 UART4:FRONT UART5:Top UART6:Debugger"
- note added: "WRITER"
- note added: "buzzer"
- moved on the sheet: BZ1, C1, J1, J7, J8, Q1, R1, R10, R11, R12, R2, R3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
