File: 02-top/02-top.kicad_sch (KiCad schematic)
At the start: 30 parts, among them J1 WRITER CONN, J2 ToMAIN, J3 PWR CONN, J4 servo, U1 STM32F446RETx

Commit message: line...
Parts:
- removed J2: ToMAIN, Connector_JST:JST_XH_B4B-XH-A_1x04_P2.50mm_Vertical, symbol Connector_Generic:Conn_01x04
- added C7, C8: 10u, symbol Device:C
- added C9: 47u, symbol Device:C
- added J10: servo6, symbol Connector_Generic:Conn_01x03
- added J11: servo7, symbol Connector_Generic:Conn_01x03
- added J12: servo8, symbol Connector_Generic:Conn_01x03
- added J13: servo9, symbol Connector_Generic:Conn_01x03
- added J14: servo10, symbol Connector_Generic:Conn_01x03
- added J15: servo11, symbol Connector_Generic:Conn_01x03
- added J16: servo12, symbol Connector_Generic:Conn_01x03
- added J17: servo13, symbol Connector_Generic:Conn_01x03
- added J18: servo14, symbol Connector_Generic:Conn_01x03
- added J19: servo15, symbol Connector_Generic:Conn_01x03
- added J2: ToMAIN, symbol Connector_Generic:Conn_02x04_Counter_Clockwise
- added J20: CAM1, Connector_JST:JST_XH_B4B-XH-A_1x04_P2.50mm_Vertical, symbol Connector_Generic:Conn_01x04
- added J21: CAM2, Connector_JST:JST_XH_B4B-XH-A_1x04_P2.50mm_Vertical, symbol Connector_Generic:Conn_01x04
- added J22: CAM3, Connector_JST:JST_XH_B4B-XH-A_1x04_P2.50mm_Vertical, symbol Connector_Generic:Conn_01x04
- added J5: servo1, symbol Connector_Generic:Conn_01x03
- added J6: servo2, symbol Connector_Generic:Conn_01x03
- added J7: servo3, symbol Connector_Generic:Conn_01x03
- added J8: servo4, symbol Connector_Generic:Conn_01x03
- added J9: servo5, symbol Connector_Generic:Conn_01x03
- added R10, R11, R12, R13, R14, R15, R16, R17, R18, R19, R20, R21, R22, R23, R24, R25: 220, symbol Device:R
- added R2, R3, R4, R5, R6, R7, R8, R9: 10k, symbol Device:R
- added U4: PCA9685PW, Package_SO:TSSOP-28_4.4x9.7mm_P0.65mm, symbol Driver_LED:PCA9685PW
- added U5: ~, symbol XIAO:XIAO_ESP32C3
- J4: value servo -> servo0
Connections:
- net +3V3: now also C7.1, U4.28 (VDD)
- net +5V: now also C8.1, C9.1, J10.2 (Pin_2), J11.2 (Pin_2), J12.2 (Pin_2), J13.2 (Pin_2), J14.2 (Pin_2), J15.2 (Pin_2), J16.2 (Pin_2), J17.2 (Pin_2), J18.2 (Pin_2), J19.2 (Pin_2), J20.2 (Pin_2), J21.2 (Pin_2), J22.2 (Pin_2), J5.2 (Pin_2), J6.2 (Pin_2), J7.2 (Pin_2), J8.2 (Pin_2), J9.2 (Pin_2), U5.14 (5V)
- net GND: now also C7.2, C8.2, C9.2, J10.1 (Pin_1), J11.1 (Pin_1), J12.1 (Pin_1), J13.1 (Pin_1), J14.1 (Pin_1), J15.1 (Pin_1), J16.1 (Pin_1), J17.1 (Pin_1), J18.1 (Pin_1), J19.1 (Pin_1), J2.1 (Pin_1), J2.8 (Pin_8), J20.1 (Pin_1), J21.1 (Pin_1), J22.1 (Pin_1), J5.1 (Pin_1), J6.1 (Pin_1), J7.1 (Pin_1), J8.1 (Pin_1), J9.1 (Pin_1), R2.2, R3.2, R4.2, R5.2, R6.2, R7.2, R8.2, R9.2, U4.14 (VSS), U5.13 (GND)
- net I2C2_SCL: now also U4.26 (SCL)
- net I2C2_SDA: now also U1.55 (PB3), U4.27 (SDA); no longer U1.53 (PC12)
- net LED_L: now also J2.5 (Pin_5)
- net LED_R: now also J2.4 (Pin_4)
- net UART2_RX: now also U1.17 (PA3), J2.3 (Pin_3)
- net UART2_TX: now also U1.16 (PA2), J2.2 (Pin_2)
- net servo1: now also J5.3 (Pin_3), R11.2; no longer J4.3 (Pin_3)
- net UART4_TX: now reaches U1.14 (PA0)
- net UART4_TX: now also J21.3 (Pin_3)
- net UART4_RX: now reaches U1.15 (PA1)
- net UART4_RX: now also J21.4 (Pin_4)
- net UART3_RX: now reaches U1.25 (PC5)
- net UART3_RX: now also J20.4 (Pin_4)
- net UART3_TX: now reaches U1.51 (PC10)
- net UART3_TX: now also J20.3 (Pin_3)
- net UART5_RX: now reaches U1.54 (PD2)
- net UART5_RX: now also J22.4 (Pin_4)
- new net: R4.1, U4.1 (A0)
- new net: R22.1, U4.19 (LED12)
- new net: R6.1, U4.3 (A2)
- new net: R18.1, U4.15 (LED8)
- new net: R7.1, U4.4 (A3)
- new net: R5.1, U4.2 (A1)
- new net: R11.1, U4.7 (LED1)
- new net: R23.1, U4.20 (LED13)
- new net: R14.1, U4.10 (LED4)
- new net: R15.1, U4.11 (LED5)
- new net: R16.1, U4.12 (LED6)
- new net: R17.1, U4.13 (LED7)
- new net: R19.1, U4.16 (LED9)
- new net: R20.1, U4.17 (LED10)
- new net: R21.1, U4.18 (LED11)
- new net: R24.1, U4.21 (LED14)
- new net: R25.1, U4.22 (LED15)
- new net: R3.1, U4.23 (~{OE})
- new net: R9.1, U4.24 (A5)
- new net: R2.1, U4.25 (EXTCLK)
- new net: R8.1, U4.5 (A4)
- new net: R10.1, U4.6 (LED0)
- new net: R12.1, U4.8 (LED2)
- new net: R13.1, U4.9 (LED3)
- new net C3_RX: J2.6 (Pin_6)
- new net C3_TX: J2.7 (Pin_7)
- new net UART5_TX: J22.3 (Pin_3), U1.53 (PC12)
- new net servo0: J4.3 (Pin_3), R10.2
- new net servo10: J14.3 (Pin_3), R20.2
- new net servo11: J15.3 (Pin_3), R21.2
- new net servo12: J16.3 (Pin_3), R22.2
- new net servo13: J17.3 (Pin_3), R23.2
- new net servo14: J18.3 (Pin_3), R24.2
- new net servo15: J19.3 (Pin_3), R25.2
- new net servo2: J6.3 (Pin_3), R12.2
- new net servo3: J7.3 (Pin_3), R13.2
- new net servo4: J8.3 (Pin_3), R14.2
- new net servo5: J9.3 (Pin_3), R15.2
- new net servo6: J10.3 (Pin_3), R16.2
- new net servo7: J11.3 (Pin_3), R17.2
- new net servo8: J12.3 (Pin_3), R18.2
- new net servo9: J13.3 (Pin_3), R19.2
- no-connect marks 4 -> 5
Other:
- company: (none) -> tuton
- title: (none) -> 02-top
- moved on the sheet: C1, C2, D1, D10, D11, D12, D13, D14, D15, D16, D2, D3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

Commit message: いっぱい増えた
Other:
- moved on the sheet: C3, C4, C5, C6, J1, U2, U3, U5

Commit message: わああ
Parts:
- removed C1: 100n, symbol Device:C
- removed C2: 4.7u, symbol Device:C
- removed C3, C4, C7, C8: 10u, symbol Device:C
- removed C5: 0.33u, symbol Device:C
- removed C6: 100u, symbol Device:C
- removed C9: 47u, symbol Device:C
- removed D10, D11, D12, D13, D14, D15, D16, D9: WS2812B, LED_SMD:LED_WS2812B_PLCC4_5.0x5.0mm_P3.2mm, symbol LED:WS2812B
- removed J1: WRITER CONN, Connector_PinHeader_2.54mm:PinHeader_2x04_P2.54mm_Vertical, symbol Connector_Generic:Conn_02x04_Counter_Clockwise
- removed J10: servo6, symbol Connector_Generic:Conn_01x03
- removed J11: servo7, symbol Connector_Generic:Conn_01x03
- removed J12: servo8, symbol Connector_Generic:Conn_01x03
- removed J13: servo9, symbol Connector_Generic:Conn_01x03
- removed J14: servo10, symbol Connector_Generic:Conn_01x03
- removed J15: servo11, symbol Connector_Generic:Conn_01x03
- removed J16: servo12, symbol Connector_Generic:Conn_01x03
- removed J17: servo13, symbol Connector_Generic:Conn_01x03
- removed J18: servo14, symbol Connector_Generic:Conn_01x03
- removed J19: servo15, symbol Connector_Generic:Conn_01x03
- removed J2: ToMAIN, symbol Connector_Generic:Conn_02x04_Counter_Clockwise
- removed J20: CAM1, Connector_JST:JST_XH_B4B-XH-A_1x04_P2.50mm_Vertical, symbol Connector_Generic:Conn_01x04
- removed J21: CAM2, Connector_JST:JST_XH_B4B-XH-A_1x04_P2.50mm_Vertical, symbol Connector_Generic:Conn_01x04
- removed J22: CAM3, Connector_JST:JST_XH_B4B-XH-A_1x04_P2.50mm_Vertical, symbol Connector_Generic:Conn_01x04
- removed J3: PWR CONN, symbol Connector_Generic:Conn_01x02
- removed J4: servo0, symbol Connector_Generic:Conn_01x03
- removed J5: servo1, symbol Connector_Generic:Conn_01x03
- removed J6: servo2, symbol Connector_Generic:Conn_01x03
- removed J7: servo3, symbol Connector_Generic:Conn_01x03
- removed J8: servo4, symbol Connector_Generic:Conn_01x03
- removed J9: servo5, symbol Connector_Generic:Conn_01x03
- removed R10, R11, R12, R13, R14, R15, R16, R17, R18, R19, R20, R21, R22, R23, R24, R25: 220, symbol Device:R
- removed R5, R6, R7, R8, R9: 10k, symbol Device:R
- removed U1: STM32F446RETx, Package_QFP:LQFP-64_10x10mm_P0.5mm, symbol MCU_ST_STM32F4:STM32F446RETx
- removed U2: ~, Package_TO_SOT_SMD:SOT-223-6, symbol JLCPCB_items:TPS7A4533DCQR
- removed U3: ~, Package_TO_SOT_SMD:TO-252-3_TabPin2, symbol JLCPCB_items:BA50BC0FP
- removed U4: PCA9685PW, Package_SO:TSSOP-28_4.4x9.7mm_P0.65mm, symbol Driver_LED:PCA9685PW
- removed U5: ~, symbol XIAO:XIAO_ESP32C3
- added J1: ToTop, Connector_JST:JST_XH_S4B-XH-A_1x04_P2.50mm_Horizontal, symbol Connector_Generic:Conn_01x04
- added J2: SSD1306, Connector_PinHeader_2.54mm:PinHeader_1x04_P2.54mm_Vertical, symbol Connector_Generic:Conn_01x04
- added SW1, SW2, SW3: SW_Push, Button_Switch_THT:SW_PUSH-12mm, symbol Switch:SW_Push
- added SW4: SW_SPDT, Connector_PinHeader_2.54mm:PinHeader_1x03_P2.54mm_Vertical, symbol Switch:SW_SPDT
- added U1: ~, XIAO:XIAO_Board, symbol XIAO:XIAO_ESP32C3
- R1: footprint Resistor_SMD:R_0805_2012Metric -> Resistor_THT:R_Axial_DIN0207_L6.3mm_D2.5mm_P10.16mm_Horizontal; LCSC C17414 -> (none)
- R2, R3, R4: footprint (none) -> Resistor_THT:R_Axial_DIN0207_L6.3mm_D2.5mm_P10.16mm_Horizontal
Connections:
- net BOOT0 is gone; now on net +3V3: R1.1
- net +3V3: now also R2.1, R3.1, R4.1, J2.2 (Pin_2), U1.12 (3V3)
- net +5V: now also J1.1 (Pin_1), U1.14 (5V)
- net GND: now also J1.4 (Pin_4), J2.1 (Pin_1), SW1.2, SW2.2, SW3.2, SW4.1 (A), U1.13 (GND); no longer R1.2, R2.2, R3.2, R4.2
- net UART5_RX: now also J1.2 (Pin_2), U1.7 (D6)
- net UART5_TX: now also J1.3 (Pin_3), U1.8 (D7)
- net LED_R renamed WS2812B
- net WS2812B: now also U1.4 (D3)
- new net I2C_SCL: J2.3 (Pin_3), U1.6 (D5)
- new net I2C_SDA: J2.4 (Pin_4), U1.5 (D4)
- new net SW: R4.2, SW4.2 (B), U1.3 (D2)
- new net SW1: R1.2, SW1.1, U1.11 (D10)
- new net SW2: R2.2, SW2.1, U1.10 (D9)
- new net SW3: R3.2, SW3.1, U1.9 (D8)
- no-connect marks 5 -> 4
Other:
- note added: "ESPじゃなくてRP2040です"
