File: 03-front/03-front.kicad_sch (KiCad schematic)
At the start: 13 parts, among them J1 Conn_01x10

Commit message: 全国行きたかった
Parts:
- added D1: LED, LED_THT:LED_D5.0mm, symbol Device:LED
- added R4: 100, Resistor_SMD:R_0805_2012Metric, symbol Device:R
- R1, R3, R5, R6, R9: value 100 -> 105; footprint (none) -> Resistor_SMD:R_0603_1608Metric
- R2: footprint (none) -> Resistor_SMD:R_1206_3216Metric
- U1, U2, U3, U4, U5: footprint Akiduki:RPR220 -> Akiduki:LBR127HLD
Connections:
- net +3V3: now also R4.2
- net GND: now also J1.3 (Pin_3), J1.4 (Pin_4), J1.5 (Pin_5), J1.6 (Pin_6), D1.1 (K)
- new net: D1.2 (A), R4.1
- no-connect marks 4 -> 0
Changed lines of the file:
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@@
 (kicad_sch (version 20230121) (generator eeschema)
   (paper "A4")
+  (junction (at 125.73 86.36) (diameter 0) (color 0 0 0 0)
+  )
   (junction (at 76.2 88.9) (diameter 0) (color 0 0 0 0)
   )
   (junction (at 76.2 48.26) (diameter 0) (color 0 0 0 0)
   )
+  (junction (at 125.73 88.9) (diameter 0) (color 0 0 0 0)
+  )
+  (junction (at 125.73 91.44) (diameter 0) (color 0 0 0 0)
+  )
   (junction (at 125.73 76.2) (diameter 0) (color 0 0 0 0)
   )
@@
   (junction (at 76.2 130.81) (diameter 0) (color 0 0 0 0)
   )
+  (junction (at 125.73 83.82) (diameter 0) (color 0 0 0 0)
+  )
   (junction (at 76.2 68.58) (diameter 0) (color 0 0 0 0)
   )
-  (no_connect (at 124.46 86.36))
-  (no_connect (at 124.46 83.82))
-  (no_connect (at 124.46 81.28))
-  (no_connect (at 124.46 88.9))
   (wire (pts (xy 76.2 48.26) (xy 80.01 48.26))
     (stroke (width 0) (type default))
@@
     (stroke (width 0) (type default))
   )
+  (wire (pts (xy 125.73 86.36) (xy 125.73 88.9))
+    (stroke (width 0) (type default))
+  )
   (wire (pts (xy 120.65 46.99) (xy 120.65 53.34))
     (stroke (width 0) (type default))
@@
     (stroke (width 0) (type default))
   )
-  (wire (pts (xy 124.46 86.36) (xy 125.73 86.36))
-    (stroke (width 0) (type default))
-  )
   (wire (pts (xy 76.2 142.24) (xy 76.2 130.81))
     (stroke (width 0) (type default))
@@
     (stroke (width 0) (type default))
   )
-  (wire (pts (xy 124.46 83.82) (xy 125.73 83.82))
-    (stroke (width 0) (type default))
-  )
   (wire (pts (xy 39.37 48.26) (xy 41.91 48.26))
     (stroke (width 0) (type default))
@@
     (stroke (width 0) (type default))
   )
-  (wire (pts (xy 124.46 88.9) (xy 125.73 88.9))
+  (wire (pts (xy 150.495 64.77) (xy 157.48 64.77))
     (stroke (width 0) (type default))
   )
@@
     (stroke (width 0) (type default))
   )
+  (wire (pts (xy 125.73 83.82) (xy 125.73 86.36))
+    (stroke (width 0) (type default))
+  )
   (wire (pts (xy 120.65 99.06) (xy 125.73 99.06))
     (stroke (width 0) (type default))
@@
     (stroke (width 0) (type default))
   )
+  (wire (pts (xy 125.73 81.28) (xy 125.73 83.82))
+    (stroke (width 0) (type default))
+  )
+  (wire (pts (xy 125.73 88.9) (xy 125.73 91.44))
+    (stroke (width 0) (type default))
+  )
   (wire (pts (xy 68.58 142.24) (xy 76.2 142.24))
-    (stroke (width 0) (type default))
-  )
-  (wire (pts (xy 124.46 81.28) (xy 125.73 81.28))
     (stroke (width 0) (type default))
   )
@@
       (effects (font (size 1.27 1.27)))
     )
-    (property "Footprint" "Akiduki:RPR220" (at 53.34 45.72 0)
+    (property "Footprint" "Akiduki:LBR127HLD" (at 53.34 45.72 0)
       (effects (font (size 1.27 1.27)) hide)
     )
@@
       (effects (font (size 1.27 1.27)))
     )
-    (property "Footprint" "" (at 83.82 46.482 90)
+    (property "Footprint" "Resistor_SMD:R_1206_3216Metric" (at 83.82 46.482 90)
       (effects (font (size 1.27 1.27)) hide)
     )
@@
       (effects (font (size 1.27 1.27)))
     )
-    (property "Value" "100" (at 39.37 45.72 90)
-      (effects (font (size 1.27 1.27)))
-    )
-    (property "Footprint" "" (at 35.56 46.482 90)
+    (property "Value" "105" (at 39.37 45.72 90)
+      (effects (font (size 1.27 1.27)))
+    )
+    (property "Footprint" "Resistor_SMD:R_0603_1608Metric" (at 35.56 46.482 90)
       (effects (font (size 1.27 1.27)) hide)
     )
@@
       (effects (font (size 1.27 1.27)))
     )
-    (property "Footprint" "Akiduki:RPR220" (at 53.34 128.27 0)
+    (property "Footprint" "Akiduki:LBR127HLD" (at 53.34 128.27 0)
       (effects (font (size 1.27 1.27)) hide)
     )
@@
         (path "/543d3245-91c2-446e-ad4e-0da5ad737f87"
           (reference "#PWR025") (unit 1)
+        )
+      )
+    )
+  )
+  (symbol (lib_id "power:GND") (at 150.495 64.77 0) (unit 1)
+    (in_bom yes) (on_board yes) (dnp no) (fields_autoplaced)
+    (property "Reference" "#PWR08" (at 150.495 71.12 0)
+      (effects (font (size 1.27 1.27)) hide)
+    )
+    (property "Value" "GND" (at 150.495 69.85 0)
+      (effects (font (size 1.27 1.27)))
+    )
+    (property "Footprint" "" (at 150.495 64.77 0)
+      (effects (font (size 1.27 1.27)) hide)
+    )
+    (property "Datasheet" "" (at 150.495 64.77 0)
+      (effects (font (size 1.27 1.27)) hide)
+    )
+    (pin "1")
+    (instances
+      (project "03-front"
+        (path "/543d3245-91c2-446e-ad4e-0da5ad737f87"
+          (reference "#PWR08") (unit 1)
         )
       )
@@
       (effects (font (size 1.27 1.27)))
     )
-    (property "Value" "100" (at 39.37 106.68 90)
-      (effects (font (size 1.27 1.27)))
-    )
-    (property "Footprint" "" (at 35.56 107.442 90)
+    (property "Value" "105" (at 39.37 106.68 90)
+      (effects (font (size 1.27 1.27)))
+    )
+    (property "Footprint" "Resistor_SMD:R_0603_1608Metric" (at 35.56 107.442 90)
       (effects (font (size 1.27 1.27)) hide)
     )
@@
       (effects (font (size 1.27 1.27)))
     )
-    (property "Value" "100" (at 39.37 86.36 90)
-      (effects (font (size 1.27 1.27)))
-    )
-    (property "Footprint" "" (at 35.56 87.122 90)
+    (property "Value" "105" (at 39.37 86.36 90)
+      (effects (font (size 1.27 1.27)))
+    )
+    (property "Footprint" "Resistor_SMD:R_0603_1608Metric" (at 35.56 87.122 90)
       (effects (font (size 1.27 1.27)) hide)
     )
@@
       (effects (font (size 1.27 1.27)))
     )
-    (property "Value" "100" (at 39.37 128.27 90)
-      (effects (font (size 1.27 1.27)))
-    )
-    (property "Footprint" "" (at 35.56 129.032 90)
+    (property "Value" "105" (at 39.37 128.27 90)
+      (effects (font (size 1.27 1.27)))
+    )
+    (property "Footprint" "Resistor_SMD:R_0603_1608Metric" (at 35.56 129.032 90)
       (effects (font (size 1.27 1.27)) hide)
     )
@@
       (effects (font (size 1.27 1.27)))
     )
-    (property "Value" "100" (at 39.37 66.04 90)
-      (effects (font (size 1.27 1.27)))
-    )
-    (property "Footprint" "" (at 35.56 66.802 90)
+    (property "Value" "105" (at 39.37 66.04 90)
+      (effects (font (size 1.27 1.27)))
+    )
+    (property "Footprint" "Resistor_SMD:R_0603_1608Metric" (at 35.56 66.802 90)
       (effects (font (size 1.27 1.27)) hide)
     )
@@
       (effects (font (size 1.27 1.27)))
     )
-    (property "Footprint" "Akiduki:RPR220" (at 53.34 86.36 0)
+    (property "Footprint" "Akiduki:LBR127HLD" (at 53.34 86.36 0)
       (effects (font (size 1.27 1.27)) hide)
     )
@@
       (effects (font (size 1.27 1.27)))
     )
-    (property "Footprint" "Akiduki:RPR220" (at 53.34 106.68 0)
+    (property "Footprint" "Akiduki:LBR127HLD" (at 53.34 106.68 0)
       (effects (font (size 1.27 1.27)) hide)
     )
@@
     )
   )
+  (symbol (lib_id "Device:R") (at 168.91 64.77 90) (unit 1)
+    (in_bom yes) (on_board yes) (dnp no) (fields_autoplaced)
+    (property "Reference" "R4" (at 168.91 58.42 90)
+      (effects (font (size 1.27 1.27)))
+    )
+    (property "Value" "100" (at 168.91 60.96 90)
+      (effects (font (size 1.27 1.27)))
+    )
+    (property "Footprint" "Resistor_SMD:R_0805_2012Metric" (at 168.91 66.548 90)
+      (effects (font (size 1.27 1.27)) hide)
+    )
+    (property "Datasheet" "~" (at 168.91 64.77 0)
+      (effects (font (size 1.27 1.27)) hide)
+    )
+    (pin "1")
+    (pin "2")
+    (instances
+      (project "03-front"
+        (path "/543d3245-91c2-446e-ad4e-0da5ad737f87"
+          (reference "R4") (unit 1)
+        )
+      )
+    )
+  )
   (symbol (lib_id "S11059:S11059") (at 123.19 41.91 0) (unit 1)
     (in_bom yes) (on_board yes) (dnp no) (fields_autoplaced)
@@
     )
   )
+  (symbol (lib_id "Device:LED") (at 161.29 64.77 0) (unit 1)
+    (in_bom yes) (on_board yes) (dnp no) (fields_autoplaced)
+    (property "Reference" "D1" (at 159.7025 58.42 0)
+      (effects (font (size 1.27 1.27)))
+    )
+    (property "Value" "LED" (at 159.7025 60.96 0)
+      (effects (font (size 1.27 1.27)))
+    )
+    (property "Footprint" "LED_THT:LED_D5.0mm" (at 161.29 64.77 0)
+      (effects (font (size 1.27 1.27)) hide)
+    )
+    (property "Datasheet" "~" (at 161.29 64.77 0)
+      (effects (font (size 1.27 1.27)) hide)
+    )
+    (pin "2")
+    (pin "1")
+    (instances
+      (project "03-front"
+        (path "/543d3245-91c2-446e-ad4e-0da5ad737f87"
+          (reference "D1") (unit 1)
+        )
+      )
+    )
+  )
   (symbol (lib_id "akiduki:LBR127HLD") (at 53.34 66.04 0) (unit 1)
     (in_bom yes) (on_board yes) (dnp no) (fields_autoplaced)
@@
       (effects (font (size 1.27 1.27)))
     )
-    (property "Footprint" "Akiduki:RPR220" (at 53.34 66.04 0)
+    (property "Footprint" "Akiduki:LBR127HLD" (at 53.34 66.04 0)
       (effects (font (size 1.27 1.27)) hide)
     )
@@
         )
       )
+    )
+  )
+  (symbol (lib_id "power:+3V3") (at 172.72 64.77 270) (unit 1)
+    (in_bom yes) (on_board yes) (dnp no) (fields_autoplaced)
+    (property "Reference" "#PWR015" (at 168.91 64.77 0)
+      (effects (font (size 1.27 1.27)) hide)
+    )
+    (property "Value" "+3V3" (at 176.53 64.77 90)
+      (effects (font (size 1.27 1.27)) (justify left))
+    )
+    (property "Footprint" "" (at 172.72 64.77 0)
+      (effects (font (size 1.27 1.27)) hide)
+    )
+    (property "Datasheet" "" (at 172.72 64.77 0)
+      (effects (font (size 1.27 1.27)) hide)
+    )
+    (pin "1")
+    (instances
+      (project "03-front"
+        (path "/543d3245-91c2-446e-ad4e-0da5ad737f87"
+          (reference "#PWR015") (unit 1)
+        )
+      )

Commit message: がんばる
Parts:
- R1, R3, R5, R6, R9: LCSC (none) -> C128061
- R2: LCSC (none) -> C138242
- R4: LCSC (none) -> C304103
Changed lines of the file:
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@@
+      (effects (font (size 1.27 1.27)) hide)
+    )
+    (property "LCSC" "" (at 53.34 45.72 0)
       (effects (font (size 1.27 1.27)) hide)
     )
@@
       (effects (font (size 1.27 1.27)) hide)
     )
+    (property "LCSC" "C138242" (at 83.82 48.26 0)
+      (effects (font (size 1.27 1.27)) hide)
+    )
     (pin "2")
     (pin "1")
@@
       (effects (font (size 1.27 1.27)) hide)
     )
+    (property "LCSC" "C128061" (at 35.56 48.26 0)
+      (effects (font (size 1.27 1.27)) hide)
+    )
     (pin "2")
     (pin "1")
@@
     )
     (property "Datasheet" "" (at 53.34 128.27 0)
+      (effects (font (size 1.27 1.27)) hide)
+    )
+    (property "LCSC" "" (at 53.34 128.27 0)
       (effects (font (size 1.27 1.27)) hide)
     )
@@
       (effects (font (size 1.27 1.27)) hide)
     )
+    (property "LCSC" "C128061" (at 35.56 109.22 0)
+      (effects (font (size 1.27 1.27)) hide)
+    )
     (pin "2")
     (pin "1")
@@
       (effects (font (size 1.27 1.27)) hide)
     )
+    (property "LCSC" "C128061" (at 35.56 88.9 0)
+      (effects (font (size 1.27 1.27)) hide)
+    )
     (pin "2")
     (pin "1")
@@
       (effects (font (size 1.27 1.27)) hide)
     )
+    (property "LCSC" "C128061" (at 35.56 130.81 0)
+      (effects (font (size 1.27 1.27)) hide)
+    )
     (pin "2")
     (pin "1")
@@
       (effects (font (size 1.27 1.27)) hide)
     )
+    (property "LCSC" "C128061" (at 35.56 68.58 0)
+      (effects (font (size 1.27 1.27)) hide)
+    )
     (pin "2")
     (pin "1")
@@
     )
     (property "Datasheet" "" (at 53.34 86.36 0)
+      (effects (font (size 1.27 1.27)) hide)
+    )
+    (property "LCSC" "" (at 53.34 86.36 0)
       (effects (font (size 1.27 1.27)) hide)
     )
@@
     )
     (property "Datasheet" "~" (at 130.81 86.36 0)
+      (effects (font (size 1.27 1.27)) hide)
+    )
+    (property "LCSC" "" (at 130.81 86.36 0)
       (effects (font (size 1.27 1.27)) hide)
     )
@@
       (effects (font (size 1.27 1.27)) hide)
     )
+    (property "LCSC" "" (at 53.34 106.68 0)
+      (effects (font (size 1.27 1.27)) hide)
+    )
     (pin "2")
     (pin "1")
@@
       (effects (font (size 1.27 1.27)) hide)
     )
+    (property "LCSC" "C304103" (at 168.91 64.77 0)
+      (effects (font (size 1.27 1.27)) hide)
+    )
     (pin "1")
     (pin "2")
@@
       (effects (font (size 1.27 1.27)) hide)
     )
+    (property "LCSC" "" (at 123.19 41.91 0)
+      (effects (font (size 1.27 1.27)) hide)
+    )
     (pin "1")
     (pin "4")
@@
       (effects (font (size 1.27 1.27)) hide)
     )
+    (property "LCSC" "" (at 161.29 64.77 0)
+      (effects (font (size 1.27 1.27)) hide)
+    )
     (pin "2")
     (pin "1")
@@
       (effects (font (size 1.27 1.27)) hide)
     )
+    (property "LCSC" "" (at 53.34 66.04 0)
+      (effects (font (size 1.27 1.27)) hide)
+    )

Commit message: いっぱい増えた
Parts:
- removed D1: LED, LED_THT:LED_D5.0mm, symbol Device:LED
- removed J1: Conn_01x10, Connector_PinHeader_2.54mm:PinHeader_1x10_P2.54mm_Horizontal, symbol Connector_Generic:Conn_01x10
- removed R3, R5, R6, R9: 105, Resistor_SMD:R_0603_1608Metric, symbol Device:R
- removed R4: 100, Resistor_SMD:R_0805_2012Metric, symbol Device:R
- removed U1, U2, U3, U4, U5: ~, Akiduki:LBR127HLD, symbol akiduki:LBR127HLD
- removed U6: ~, S11059:S11059, symbol S11059:S11059
- added C1, C3, C4, C5, C6, C8, C9: 100n, Capacitor_SMD:C_0402_1005Metric, symbol Device:C
- added C10: 1u, Capacitor_SMD:C_0402_1005Metric, symbol Device:C
- added C2, C7: 4.7u, Capacitor_SMD:C_0402_1005Metric, symbol Device:C
- added FB1: FerriteBead, Resistor_SMD:R_0805_2012Metric, symbol Device:FerriteBead
- added J1: WRITER CONN, Connector_PinHeader_2.54mm:PinHeader_2x04_P2.54mm_Vertical, symbol Connector_Generic:Conn_02x04_Counter_Clockwise
- added J10, J11, J12, J8, J9: VL53L0X_X, symbol Connector_Generic:Conn_01x01
- added J13: ToMAIN, Connector_PinHeader_2.54mm:PinHeader_1x04_P2.54mm_Vertical, symbol Connector_Generic:Conn_01x04
- added J2: ST-LINK, Connector_PinHeader_2.54mm:PinHeader_1x04_P2.54mm_Vertical, symbol Connector_Generic:Conn_01x04
- added J3, J4, J5, J6, J7: VL53L0X, symbol Connector_Generic:Conn_01x04
- added U1: STM32F446RETx, Package_QFP:LQFP-64_10x10mm_P0.5mm, symbol MCU_ST_STM32F4:STM32F446RETx
- R1: value 105 -> 10k; LCSC C128061 -> C137819
- R2: value 1k -> 10k; footprint Resistor_SMD:R_1206_3216Metric -> Resistor_SMD:R_0603_1608Metric; LCSC C138242 -> C137819
Connections:
- net photo1 is gone; now on net GND: R2.2
- net +3V3: now also C3.2, C4.2, C5.2, C6.2, C7.1, C8.2, FB1.1, J1.8 (Pin_8), J3.1 (Pin_1), J4.1 (Pin_1), J5.1 (Pin_1), J6.1 (Pin_1), J7.1 (Pin_1), U1.1 (VBAT), U1.19 (VDD), U1.32 (VDD), U1.48 (VDD), U1.64 (VDD); no longer R2.1
- net GND: now also C1.1, C10.1, C2.2, C3.1, C4.1, C5.1, C6.1, C7.2, C8.1, C9.1, J1.6 (Pin_6), J2.4 (Pin_4), J3.2 (Pin_2), J4.2 (Pin_2), J5.2 (Pin_2), J6.2 (Pin_2), J7.2 (Pin_2), U1.12 (VSSA), U1.18 (VSS), U1.31 (VSS), U1.47 (VSS), U1.63 (VSS)
- net BOOT0: now reaches R1.1
- net BOOT0: now also J1.5 (Pin_5), U1.60 (BOOT0)
- new net: R2.1, U1.28 (PB2)
- new net: C10.2, C9.2, FB1.2, U1.13 (VDDA)
- new net: C2.1, U1.30 (VCAP_1)
- new net I2C1_SCL: J3.3 (Pin_3), J4.3 (Pin_3), J5.3 (Pin_3), J6.3 (Pin_3), J7.3 (Pin_3), U1.58 (PB6)
- new net I2C1_SDA: J3.4 (Pin_4), J4.4 (Pin_4), J5.4 (Pin_4), J6.4 (Pin_4), J7.4 (Pin_4), U1.59 (PB7)
- new net I2C2_SCL: U1.29 (PB10)
- new net I2C2_SDA: U1.53 (PC12)
- new net NRST: C1.2, J1.3 (Pin_3), J2.3 (Pin_3), U1.7 (NRST)
- new net SWCLK: J2.1 (Pin_1), U1.49 (PA14)
- new net SWDIO: J2.2 (Pin_2), U1.46 (PA13)
- new net UART1_RX: J1.2 (Pin_2), U1.43 (PA10)
- new net UART1_TX: J1.4 (Pin_4), U1.42 (PA9)
- new net UART2_RX: U1.17 (PA3)
- new net UART2_TX: U1.16 (PA2)
- new net UART3_RX: U1.25 (PC5)
- new net UART3_TX: U1.51 (PC10)
- new net UART4_RX: U1.15 (PA1)
- new net UART4_TX: U1.14 (PA0)
- no-connect marks 0 -> 2

Commit message: わああ
Parts:
- removed J10, J11, J12, J8, J9: VL53L0X_X, symbol Connector_Generic:Conn_01x01
- removed J13: ToMAIN, Connector_PinHeader_2.54mm:PinHeader_1x04_P2.54mm_Vertical, symbol Connector_Generic:Conn_01x04
- removed J3, J4, J5, J6, J7: VL53L0X, symbol Connector_Generic:Conn_01x04
- added D1, D10, D11, D12, D2, D3, D4, D5, D6, D7, D8, D9: WS2812B, LED_SMD:LED_WS2812B_PLCC4_5.0x5.0mm_P3.2mm, symbol LED:WS2812B
- added R3, R4: 10k, Resistor_SMD:R_0603_1608Metric, symbol Device:R
- added U2, U3, U4, U5, U6: ~, tuton:VL53L0X_horizontal, symbol tuton_module:vl53l0x_module
- added U7: ~, OpenMV:OpenMV h7, symbol OpenMV:OpenMV_h7
- C1, C3, C4, C5, C6, C8, C9: LCSC C3012377 -> C1525
- C10: LCSC C3012378 -> C52923
- C2, C7: LCSC C7472956 -> C23733
- J1: footprint Connector_PinHeader_2.54mm:PinHeader_2x04_P2.54mm_Vertical -> Connector_PinSocket_2.54mm:PinSocket_2x04_P2.54mm_Vertical
- J2: value ST-LINK -> ToMAIN; footprint Connector_PinHeader_2.54mm:PinHeader_1x04_P2.54mm_Vertical -> Connector_JST:JST_XH_B4B-XH-A_1x04_P2.50mm_Vertical
- R1, R2: LCSC C137819 -> C25804
Connections:
- net +3V3: now also R3.1, R4.2, U2.1 (3V3), U3.1 (3V3), U4.1 (3V3), U5.1 (3V3), U6.1 (3V3), U7.8 (3V3)
- net GND: now also D1.3 (VSS), D10.3 (VSS), D11.3 (VSS), D12.3 (VSS), D2.3 (VSS), D3.3 (VSS), D4.3 (VSS), D5.3 (VSS), D6.3 (VSS), D7.3 (VSS), D8.3 (VSS), D9.3 (VSS), U2.2 (GND), U3.2 (GND), U4.2 (GND), U5.2 (GND), U6.2 (GND), U7.16 (GND)
- net I2C1_SCL: now also R4.1, U2.3 (SCL), U3.3 (SCL), U4.3 (SCL), U5.3 (SCL), U6.3 (SCL)
- net I2C1_SDA: now also R3.2, U2.4 (SDA), U3.4 (SDA), U4.4 (SDA), U5.4 (SDA), U6.4 (SDA)
- net NRST: no longer J2.3 (Pin_3)
- net UART2_RX: now also J2.3 (Pin_3)
- net UART2_TX: now also J2.2 (Pin_2)
- net UART3_RX: now also U7.2 (P1)
- net UART3_TX: now also U7.1 (P0)
- net XSHUT1: now reaches U1.20 (PA4)
- net XSHUT1: now also U2.5 (XSHUT)
- net XSHUT2: now reaches U1.21 (PA5)
- net XSHUT2: now also U3.5 (XSHUT)
- net XSHUT3: now reaches U1.22 (PA6)
- net XSHUT3: now also U4.5 (XSHUT)
- net XSHUT4: now reaches U1.23 (PA7)
- net XSHUT4: now also U5.5 (XSHUT)
- net XSHUT5: now reaches U1.41 (PA8)
- net XSHUT5: now also U6.5 (XSHUT)
- net WS2812B: now reaches U1.44 (PA11)
- net WS2812B: now also D1.4 (DIN)
- net I2C2_SCL: no longer names the net of U1.29 (PB10)
- net I2C2_SDA: no longer names the net of U1.53 (PC12)
- net SWCLK: no longer names the net of U1.49 (PA14)
- net SWCLK: no longer J2.1 (Pin_1)
- net SWDIO: no longer names the net of U1.46 (PA13)
- net SWDIO: no longer J2.2 (Pin_2)
- net UART4_RX: no longer names the net of U1.15 (PA1)
- net UART4_TX: no longer names the net of U1.14 (PA0)
- new net: D7.2 (DOUT), D8.4 (DIN)
- new net: D6.2 (DOUT), D7.4 (DIN)
- new net: D5.2 (DOUT), D6.4 (DIN)
- new net: D4.2 (DOUT), D5.4 (DIN)
- new net: D8.2 (DOUT), D9.4 (DIN)
- new net: D10.4 (DIN), D9.2 (DOUT)
- new net: D2.2 (DOUT), D3.4 (DIN)
- new net: D1.2 (DOUT), D2.4 (DIN)
- new net: D3.2 (DOUT), D4.4 (DIN)
- new net: D11.2 (DOUT), D12.4 (DIN)
- new net: D10.2 (DOUT), D11.4 (DIN)
- new net +5V: D1.1 (VDD), D10.1 (VDD), D11.1 (VDD), D12.1 (VDD), D2.1 (VDD), D3.1 (VDD), D4.1 (VDD), D5.1 (VDD), D6.1 (VDD), D7.1 (VDD), D8.1 (VDD), D9.1 (VDD), J2.1 (Pin_1), U7.15 (VIN)
- no-connect marks 2 -> 60
