File: 2-KANTO/02-LINE/02-LINE.kicad_pcb (KiCad board)
At the start: 2 copper layers, 81 x 52 mm, 78 parts, among them J2 WRITER CONN, J3 Conn_01x05, U1 STM32F446RETx

Commit message: mike
Parts:
- added G***: LOGO, logo:st_logo_small, F.Cu at (169.3, 126.7)
- added G***: LOGO, logo:tuton_logo_small, F.Cu at (164.1, 126.5)
- added G***: LOGO, logo:jlcpcb_logo, F.Cu at (164.8, 130.2)
Connections:
- J2 pad 2: +3V3 -> UART1_RX
- J2 pad 3: BOOT0 -> NRST
- J2 pad 4: GND -> UART1_TX
- J2 pad 5: NRST -> BOOT0
- J2 pad 6: UART1_TX -> GND
- J2 pad 8: UART1_RX -> +3V3
Routing:
- net +3V3: track 313.4 -> 326.3 mm
- net UART1_RX: track 73.9 -> 83.5 mm
- net NRST: track 35.1 -> 39.8 mm
- net UART1_TX: track 53.1 -> 50.9 mm
- net GND: track 119.6 -> 121.4 mm, vias 77 -> 76
- net BOOT0: track 40.6 -> 39.5 mm
Other:
- board text added: "1"
- board text added: "3V3"
- board text added: "5V"
- board text added: "BOOT0"
- board text added: "GND"
- board text added: "NRST"
- board text added: "RX"
- board text added: "TX"
- board text added: "Tuton MIKE 02-LINE ver.1"
- board text added: "x"
