File: 2-KANTO/04-PWR/04-PWR.kicad_pcb (KiCad board)
At the start: 2 copper layers, 100 x 110 mm, 34 parts, among them J1 MAIN Conn, J2 voltmeter, J3 Battery, J4 OpenMV Conn, J5 Conn_01x20, J6 Conn_01x20, M1 ServoBasketLeft, M2 ServoBasketRight, M3 ServoArmLeft, M4 ServoArmRight, M5 ServoHandLeft, M6 ServoHandRight, Q1 Q_PMOS_GDS, SW1 SW_SPDT, SW2 SW_SPST, U3 RASPBERRY_PI_PICO

Commit message: mike
Parts:
- removed F2: Fuse, Akiduki:FUSE_3557-15
- removed M2: ServoBasketRight, Connector_PinHeader_2.54mm:PinHeader_1x03_P2.54mm_Horizontal
- removed RV1: R_Trim_5V, Potentiometer_THT:Potentiometer_Bourns_3006P_Horizontal
- removed RV2: R_Trim_3V3, Potentiometer_THT:Potentiometer_Bourns_3006P_Horizontal
- added C10: 10uF, Capacitor_SMD:C_0805_2012Metric, F.Cu at (124.5, 121.9)
- added C11: 10uF, Capacitor_SMD:C_0805_2012Metric, F.Cu at (102.2, 123.2)
- added C5: 100n, Capacitor_SMD:C_0402_1005Metric, F.Cu at (119.4, 65.0)
- added C6: 100n, Capacitor_SMD:C_0402_1005Metric, F.Cu at (116.8, 70.8)
- added C7: 4.7u, Resistor_SMD:R_0402_1005Metric, F.Cu at (117.9, 64.8)
- added C8: 22uF, Capacitor_SMD:C_0805_2012Metric, F.Cu at (124.0, 128.5)
- added C9: 22uF, Capacitor_SMD:C_0805_2012Metric, F.Cu at (101.6, 128.0)
- added D1: LED_GREEN, LED_SMD:LED_0805_2012Metric, F.Cu at (170.8, 54.0)
- added F1: Fuse, Akiduki:FUSE_3557-15, F.Cu at (168.9, 141.9)
- added G***: LOGO, logo:st_logo_middle, F.Cu at (145.3, 51.1)
- added G***: LOGO, logo:tuton_logo, F.Cu at (160.3, 50.3)
- added G***: LOGO, logo:jlcpcb_logo_big, F.Cu at (118.1, 50.5)
- added J7: voltmeter, Connector_JST:JST_XH_S2B-XH-A_1x02_P2.50mm_Horizontal, F.Cu at (107.9, 107.6)
- added J8: Battery, Connector_Wire:SolderWire-2sqmm_1x02_P7.8mm_D2mm_OD3.9mm, F.Cu at (151.9, 138.4)
- added M: ServoBasketRight, Connector_PinHeader_2.54mm:PinHeader_1x03_P2.54mm_Vertical, F.Cu at (92.5, 143.0)
- added R11: 680, Resistor_SMD:R_0603_1608Metric, F.Cu at (143.5, 122.7)
- added R12: 1.2k, Resistor_SMD:R_0603_1608Metric, F.Cu at (122.6, 122.1)
- added R13: 1.2k, Resistor_SMD:R_0603_1608Metric, F.Cu at (100.3, 123.1)
- added R2: 10k, Resistor_SMD:R_0603_1608Metric, F.Cu at (160.7, 79.8)
- added R3: 10k, Resistor_SMD:R_0603_1608Metric, F.Cu at (85.1, 50.3)
- added R4: 10k, Resistor_SMD:R_0603_1608Metric, F.Cu at (79.5, 149.9)
- added R5: 470, Resistor_SMD:R_0603_1608Metric, F.Cu at (170.6, 52.1)
- added R6: 10k, Resistor_SMD:R_0603_1608Metric, F.Cu at (163.8, 143.5)
- added REF**: MountingHole_3.2mm_M3, MountingHole:MountingHole_3.2mm_M3, F.Cu at (160.0, 140.0)
- added REF**: MountingHole_3.2mm_M3, MountingHole:MountingHole_3.2mm_M3, F.Cu at (80.0, 55.0)
- added REF**: MountingHole_3.2mm_M3, MountingHole:MountingHole_3.2mm_M3, F.Cu at (160.0, 60.0)
- added REF**: MountingHole_3.2mm_M3, MountingHole:MountingHole_3.2mm_M3, F.Cu at (80.0, 145.0)
- C1, C2: value 22uF -> 100n; footprint Capacitor_SMD:C_0805_2012Metric_Pad1.18x1.45mm_HandSolder -> Capacitor_SMD:C_0402_1005Metric
- C3, C4: value 10uF -> 100n; footprint Capacitor_SMD:C_1206_3216Metric_Pad1.33x1.80mm_HandSolder -> Capacitor_SMD:C_0402_1005Metric
- J1: value MAIN Conn -> PB_PIN; footprint Connector_JST:JST_XH_B8B-XH-A_1x08_P2.50mm_Vertical -> Connector_PinHeader_2.54mm:PinHeader_1x16_P2.54mm_Vertical
- J2: value voltmeter -> Conn_01x05; footprint Connector_Wire:SolderWire-0.5sqmm_1x02_P4.6mm_D0.9mm_OD2.1mm -> Connector_PinHeader_2.54mm:PinHeader_1x05_P2.54mm_Vertical
- J3: value Battery -> PA_PIN; footprint Connector_Wire:SolderWire-2sqmm_1x02_P7.8mm_D2mm_OD3.9mm -> Connector_PinHeader_2.54mm:PinHeader_1x16_P2.54mm_Vertical
- J4: value OpenMV Conn -> WRITER CONN; footprint Connector_JST:JST_XH_B4B-XH-A_1x04_P2.50mm_Vertical -> Connector_PinSocket_2.54mm:PinSocket_2x04_P2.54mm_Horizontal
- J5: value Conn_01x20 -> MAIN Conn; footprint Connector_PinHeader_2.54mm:PinHeader_1x20_P2.54mm_Vertical -> Connector_JST:JST_XH_S8B-XH-A_1x08_P2.50mm_Horizontal
- J6: value Conn_01x20 -> OpenMV Conn; footprint Connector_PinHeader_2.54mm:PinHeader_1x20_P2.54mm_Vertical -> Connector_JST:JST_XH_S4B-XH-A_1x04_P2.50mm_Horizontal
- M1: footprint Connector_PinHeader_2.54mm:PinHeader_1x03_P2.54mm_Horizontal -> Connector_PinHeader_2.54mm:PinHeader_1x03_P2.54mm_Vertical
- R1: footprint Resistor_THT:R_Axial_DIN0207_L6.3mm_D2.5mm_P10.16mm_Horizontal -> Resistor_SMD:R_0603_1608Metric
- R10: value 10k -> 1.5k; footprint Resistor_THT:R_Axial_DIN0207_L6.3mm_D2.5mm_P10.16mm_Horizontal -> Resistor_SMD:R_0603_1608Metric
- R7: value 1.2k -> 1k; footprint Resistor_THT:R_Axial_DIN0207_L6.3mm_D2.5mm_P10.16mm_Horizontal -> Resistor_SMD:R_0603_1608Metric
- R8: value 1.2k -> 330; footprint Resistor_THT:R_Axial_DIN0207_L6.3mm_D2.5mm_P10.16mm_Horizontal -> Resistor_SMD:R_0603_1608Metric
- R9: value 10k -> 10; footprint Resistor_THT:R_Axial_DIN0207_L6.3mm_D2.5mm_P10.16mm_Horizontal -> Resistor_SMD:R_0603_1608Metric
- SW1: footprint Connector_PinHeader_2.54mm:PinHeader_1x03_P2.54mm_Vertical -> Akiduki:SK-12D11VG3
- U1: value ~ -> STM32F103C8Tx; footprint Akiduki:OKL-T6-W12N-C-SMD -> Package_QFP:LQFP-48_7x7mm_P0.5mm
- U2: footprint Akiduki:OKL-T6-W12N-C-SMD -> tuton:vl53l0x_vertical
- U3: value RASPBERRY_PI_PICO -> ~; footprint Akiduki:RASPBERRY_PI_PICO -> tuton:vl53l0x_vertical
- U4: footprint tuton:vl53l0x_vertical -> Akiduki:OKL-T6-W12N-C-SMD
- U5: footprint tuton:vl53l0x_vertical -> Akiduki:OKL-T6-W12N-C-SMD; moved to F.Cu
- moved U3 128.4 mm to (83.8, 152.4), turned to 0 degrees
- moved U5 117.7 mm to (111.8, 126.8), turned to 90 degrees
- moved U2 115.0 mm to (81.3, 47.5), turned to 180 degrees
- moved J6 109.0 mm to (92.6, 109.3)
- moved H1 108.2 mm to (96.0, 150.0)
- moved J2 105.5 mm to (109.2, 73.7), turned to 180 degrees
- moved H2 98.5 mm to (96.0, 50.0)
- moved U4 96.7 mm to (134.8, 127.0), turned to 90 degrees
- moved J3 88.7 mm to (101.6, 81.3), turned to 90 degrees
- moved R1 83.2 mm to (124.0, 76.7)
- moved J5 67.5 mm to (92.7, 85.4), turned to -90 degrees
- moved C2 58.4 mm to (115.8, 69.8), turned to 90 degrees
- moved C1 58.4 mm to (117.8, 66.0), turned to 180 degrees
- moved U1 56.9 mm to (123.2, 69.8)
- moved C4 51.8 mm to (129.0, 67.0), turned to -90 degrees
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Connections:
- C1 pad 1: VDD -> +3V3
- C2 pad 1: VDD -> GND
- C2 pad 2: GND -> NRST
- C4 pad 1: +5V -> +3V3
- J1 pad 1: LoPSwitch -> Net-(J1-Pin_1)
- J1 pad 2: +3V3 -> Net-(J1-Pin_2)
- J1 pad 3: OpenMV->MAIN -> Net-(J1-Pin_3)
- J1 pad 4: MAIN->OpenMV -> Net-(J1-Pin_4)
- J1 pad 5: +5V -> Net-(J1-Pin_5)
- J1 pad 6: PWR->MAIN -> Net-(J1-Pin_6)
- J1 pad 7: MAIN->PWR -> SCL
- J1 pad 8: GND -> SDA
- J2 pad 1: VDD -> Net-(J2-Pin_1)
- J2 pad 2: GND -> Net-(J2-Pin_2)
- J3 pad 1: Net-(J3-Pin_1) -> ServoHandLeft
- J3 pad 2: GND -> ServoHandRight
- J4 pad 1: +5V -> unconnected-(J4-Pin_1-Pad1)
- J4 pad 2: OpenMV->MAIN -> UART1_RX
- J4 pad 3: MAIN->OpenMV -> NRST
- J4 pad 4: GND -> UART1_TX
- J5 pad 1: Net-(J5-Pin_1) -> LoPSwitch
- J5 pad 2: Net-(J5-Pin_2) -> +3V3
- J5 pad 3: GND -> OpenMV->MAIN
- J5 pad 4: Net-(J5-Pin_4) -> MAIN->OpenMV
- J5 pad 5: Net-(J5-Pin_5) -> +5V
- J5 pad 6: XSHUT2 -> PWR->MAIN
- J5 pad 7: XSHUT1 -> MAIN->PWR
- J6 pad 1: Net-(J6-Pin_1) -> +5V
- J6 pad 2: +5V -> OpenMV->MAIN
- J6 pad 3: GND -> MAIN->OpenMV
- J6 pad 4: Net-(J6-Pin_4) -> GND
- R1 pad 1: Net-(Q1-S) -> GND
- R1 pad 2: Net-(Q1-G) -> Net-(J1-Pin_3)
- R10 pad 1: +3V3 -> Net-(U4-Trim)
- R10 pad 2: SDA -> Net-(R10-Pad2)
- R7 pad 1: +3V3 -> Net-(U5-Trim)
- R7 pad 2: GND -> Net-(R7-Pad2)
- R8 pad 1: +5V -> Net-(R7-Pad2)
- R8 pad 2: GND -> Net-(R8-Pad2)
- R9 pad 1: SCL -> Net-(R8-Pad2)
- R9 pad 2: +3V3 -> GND
- U1 pad 1: GND -> +3V3
- U1 pad 10: unconnected-(U1-PGOOD-Pad10) -> ServoHandLeft
- U1 pad 11: unconnected-(U1-N.C.-Pad11) -> ServoHandRight
- U1 pad 12: unconnected-(U1-N.C.-Pad12) -> ServoArmLeft
- U1 pad 2: VDD -> Net-(J2-Pin_3)
- U1 pad 3: GND -> Net-(J2-Pin_2)
- U1 pad 4: +3V3 -> Net-(J2-Pin_1)
- U1 pad 5: +3V3 -> Net-(J2-Pin_5)
- U1 pad 6: Net-(U1-Trim) -> Net-(J2-Pin_4)
- U1 pad 7: GND -> NRST
- U1 pad 8: unconnected-(U1-N.C.-Pad8) -> GND
- U1 pad 9: unconnected-(U1-Sequence-Pad9) -> +3V3
- U2 pad 1: GND -> +3V3
- U2 pad 2: VDD -> GND
- U2 pad 3: GND -> SCL
- U2 pad 4: +5V -> SDA
- U2 pad 5: +5V -> XSHUT1
- U2 pad 6: Net-(U2-Trim) -> unconnected-(U2-GPIO-Pad6)
- U4 pad 1: +3V3 -> GND
- U4 pad 2: GND -> VDD
- U4 pad 3: SCL -> GND
- U4 pad 4: SDA -> +3V3
- U4 pad 5: XSHUT1 -> +3V3
- U4 pad 6: unconnected-(U4-GPIO-Pad6) -> Net-(U4-Trim)
- U5 pad 1: +3V3 -> GND
- U5 pad 2: GND -> VDD
- U5 pad 3: SCL -> GND
- U5 pad 4: SDA -> +5V
- U5 pad 5: XSHUT2 -> +5V
- U5 pad 6: unconnected-(U5-GPIO-Pad6) -> Net-(U5-Trim)
Routing:
- net +3V3: track 0.00 -> 457.4 mm, vias 0 -> 3
- net SDA: track 5.08 -> 180.5 mm, vias 0 -> 1
- net SCL: track 5.08 -> 164.1 mm, vias 0 -> 1
- net XSHUT2: track 5.08 -> 149.8 mm, vias 0 -> 2
- net GND: track 40.6 -> 138.0 mm, vias 0 -> 94
- net LoPSwitch: track 0.00 -> 88.2 mm, vias 0 -> 3
- net MAIN->PWR: track 5.08 -> 90.9 mm, vias 0 -> 4
- net ServoBasketRight: track 5.08 -> 86.6 mm, vias 0 -> 1
- net PWR->MAIN: track 5.08 -> 86.0 mm, vias 0 -> 2
- net XSHUT1: track 5.08 -> 83.4 mm, vias 0 -> 2
- net ServoHandRight: track 5.08 -> 81.2 mm, vias 0 -> 1
- net NRST: track 0.00 -> 67.2 mm, vias 0 -> 2
- net UART1_TX: track 0.00 -> 63.7 mm
- net ServoArmRight: track 5.08 -> 68.4 mm, vias 0 -> 1
- net UART1_RX: track 0.00 -> 60.6 mm
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- added copper zone on F.Cu, net +3V3
- added copper zone on F.Cu, net +5V
- added copper zone on B.Cu, net GND
- added copper zone on F.Cu, net GND
- added copper zone on F.Cu, net Net-(Q1-S)
- added copper zone on F.Cu, net VDD
Other:
- outline, holes or cut-outs redrawn
- board text added: "1"
- board text added: "3V3"
- board text added: "5V"
- board text added: "Arm"
- board text added: "BOOT"
- board text added: "Basket"
- board text added: "G"
- board text added: "G-D-S"
- board text added: "GND"
- board text added: "Hand"
- board text added: "MAIN-CAM"
- board text added: "MAIN-PWR"
- board text added: "NRST"
- board text added: "PWR SW"
- board text added: "RX"
- board text added: "S"
- board text added: "SW"
- board text added: "TX"
- board text added: "Trim"
- board text added: "Tuton MIKE 04-PWR ver.1"
- board text added: "V"
- board text added: "VBAT"
- board text added: "VDD"
- board text added: "VOLTMETER"
- board text added: "X"
- board text added: "mosfet"
- board text added: "x"
