File: 1-TOKYO/05-PWR/05-PWR.kicad_sch (KiCad schematic)
At the start: 37 parts, among them J1 Battery, J1 ToLINE, J10 5V ToMAIN, J11 Conn_01x04, J2 VOLTMETER, J3 STS3032, J4 STS3032, J5 STS3032, J6 STS3032, J9 3V3 ToMAIN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

Commit message: readme
Other:
- moved on the sheet: C1, C2, C3, C4, R1, R2, R3, R4, R5, R6, R8, U3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
