File: 1-TOKYO/09-ToF_mod/09-ToF_mod.kicad_pcb (KiCad board)
At the start: 2 copper layers, 10.7 x 13.7 mm, 12 parts, among them J1 Conn_01x04, J2 Conn_01x02, U1 VL53L0X

Commit message: 03-FRONT部品配置終わり
Parts:
- J1: footprint Connector_PinHeader_2.54mm:PinHeader_1x04_P2.54mm_Horizontal -> Connector_PinHeader_2.54mm:PinHeader_1x04_P2.54mm_Vertical
