File: 3-NAGOYA/06-UI/06-UI.kicad_sch (KiCad schematic)
At the start: 17 parts, among them J6 OpenMV Conn, SW1 SW_Push

Commit message: 01-MAIN部品配置完了
Parts:
- removed H3, H4: MountingHole, MountingHole:MountingHole_3.2mm_M3, symbol Mechanical:MountingHole
Changed lines of the file:
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@@
-    )
-  )
-  (symbol (lib_id "Mechanical:MountingHole") (at 118.745 92.075 0) (unit 1)
-    (in_bom yes) (on_board yes) (dnp no) (fields_autoplaced)
-    (property "Reference" "H4" (at 121.92 90.805 0)
-      (effects (font (size 1.27 1.27)) (justify left))
-    )
-    (property "Value" "MountingHole" (at 121.92 93.345 0)
-      (effects (font (size 1.27 1.27)) (justify left))
-    )
-    (property "Footprint" "MountingHole:MountingHole_3.2mm_M3" (at 118.745 92.075 0)
-      (effects (font (size 1.27 1.27)) hide)
-    )
-    (property "Datasheet" "~" (at 118.745 92.075 0)
-      (effects (font (size 1.27 1.27)) hide)
-    )
-    (instances
-      (project "06-UI"
-        (path "/964c7233-7aca-4175-8dc7-0604df29af02"
-          (reference "H4") (unit 1)
-        )
-      )
-      (project "03-FRONT"
-        (path "/e118ed56-ce79-44d8-8eff-a935fd9f7b40"
-          (reference "H2") (unit 1)
-        )
-      )
     )
   )
@@
         )
       )
-    )
-  )
-  (symbol (lib_id "Mechanical:MountingHole") (at 118.745 80.645 0) (unit 1)
-    (in_bom yes) (on_board yes) (dnp no) (fields_autoplaced)
-    (property "Reference" "H3" (at 121.92 79.375 0)
-      (effects (font (size 1.27 1.27)) (justify left))
-    )
-    (property "Value" "MountingHole" (at 121.92 81.915 0)
-      (effects (font (size 1.27 1.27)) (justify left))
-    )
-    (property "Footprint" "MountingHole:MountingHole_3.2mm_M3" (at 118.745 80.645 0)
-      (effects (font (size 1.27 1.27)) hide)
-    )
-    (property "Datasheet" "~" (at 118.745 80.645 0)
-      (effects (font (size 1.27 1.27)) hide)
-    )
-    (instances
-      (project "06-UI"
-        (path "/964c7233-7aca-4175-8dc7-0604df29af02"
-          (reference "H3") (unit 1)
-        )
-      )
-      (project "03-FRONT"
-        (path "/e118ed56-ce79-44d8-8eff-a935fd9f7b40"
-          (reference "H1") (unit 1)
-        )
-      )
