File: 3-NAGOYA/05-PWR/05-PWR.kicad_sch (KiCad schematic)
At the start: 23 parts, among them J7 voltmeter, J8 Battery, Q1 Q_PMOS_GDS, SW2 SW_SPST

Commit message: 03-FRONT 3Dモデル出力
Connections:
- net +7.5V is gone; now on net VDD: H1.1
Changed lines of the file:
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@@
-    )
-  )
-  (symbol (lib_id "power:+7.5V") (at 167.005 53.975 90) (unit 1)
-    (in_bom yes) (on_board yes) (dnp no) (fields_autoplaced)
-    (property "Reference" "#PWR017" (at 170.815 53.975 0)
-      (effects (font (size 1.27 1.27)) hide)
-    )
-    (property "Value" "+7.5V" (at 163.83 53.975 90)
-      (effects (font (size 1.27 1.27)) (justify left))
-    )
-    (property "Footprint" "" (at 167.005 53.975 0)
-      (effects (font (size 1.27 1.27)) hide)
-    )
-    (property "Datasheet" "" (at 167.005 53.975 0)
-      (effects (font (size 1.27 1.27)) hide)
-    )
-    (pin "1")
-    (instances
-      (project "05-PWR"
-        (path "/d90cef91-1e80-4d94-96a4-2a396e13952b"
-          (reference "#PWR017") (unit 1)
-        )
-      )
     )
   )
@@
         )
       )
+    )
+  )
+  (symbol (lib_id "power:VDD") (at 167.005 53.975 90) (unit 1)
+    (in_bom yes) (on_board yes) (dnp no) (fields_autoplaced)
+    (property "Reference" "#PWR043" (at 170.815 53.975 0)
+      (effects (font (size 1.27 1.27)) hide)
+    )
+    (property "Value" "VDD" (at 163.83 53.975 90)
+      (effects (font (size 1.27 1.27)) (justify left))
+    )
+    (property "Footprint" "" (at 167.005 53.975 0)
+      (effects (font (size 1.27 1.27)) hide)
+    )
+    (property "Datasheet" "" (at 167.005 53.975 0)
+      (effects (font (size 1.27 1.27)) hide)
+    )
+    (pin "1")
+    (instances
+      (project "04-PWR"
+        (path "/5fb95203-1119-4f22-b8d1-f5feaaf529dd"
+          (reference "#PWR043") (unit 1)
+        )
+      )
+      (project "05-PWR"
+        (path "/d90cef91-1e80-4d94-96a4-2a396e13952b"
+          (reference "#PWR017") (unit 1)
+        )
+      )

Commit message: 04-RESCUE完了。全基板あとシルクだけ
Parts:
- J7: footprint Connector_JST:JST_XH_S2B-XH-A_1x02_P2.50mm_Horizontal -> Connector_Wire:SolderWire-0.5sqmm_1x02_P4.6mm_D0.9mm_OD2.1mm
Changed lines of the file:
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@@
       (effects (font (size 1.27 1.27)) (justify left))
     )
-    (property "Footprint" "Connector_JST:JST_XH_S2B-XH-A_1x02_P2.50mm_Horizontal" (at 189.23 37.465 0)
+    (property "Footprint" "Connector_Wire:SolderWire-0.5sqmm_1x02_P4.6mm_D0.9mm_OD2.1mm" (at 189.23 37.465 0)
       (effects (font (size 1.27 1.27)) hide)
     )
