File: 3-NAGOYA/01-MAIN/01-MAIN.kicad_pcb (KiCad board)
At the start: 2 copper layers, 130 x 136 mm, 76 parts, among them J1 Front, J2 Top, J3 toLINE, J4 USB_C_Receptacle_USB2.0, J5 STS3032, J6 STS3032, J7 STS3032, J8 STS3032, Q1 2SA1015, SW1 NRST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

Commit message: 01-MAIN基板設計完了
Parts:
- D2, R8: moved to B.Cu
- moved J7 72.5 mm to (90.8, 136.1), turned to 0 degrees
- moved J5 72.2 mm to (162.1, 69.4), turned to -90 degrees
- moved C1 71.2 mm to (191.0, 108.5), turned to -90 degrees
- moved R2 69.9 mm to (191.0, 105.4), turned to -90 degrees
- moved J8 68.9 mm to (90.2, 65.5)
- moved J6 66.6 mm to (162.1, 125.8), turned to -90 degrees
- moved R6 42.0 mm to (152.1, 101.3), turned to 0 degrees
- moved C11 40.2 mm to (160.7, 95.5), turned to -90 degrees
- moved C10 39.3 mm to (159.7, 95.5), turned to -90 degrees
- moved C7 37.2 mm to (157.6, 87.6), turned to 0 degrees
- moved C3 36.3 mm to (159.7, 89.4), turned to -90 degrees
- moved FB1 36.1 mm to (162.2, 94.7), turned to -90 degrees
- moved C8 35.2 mm to (155.6, 86.4), turned to 0 degrees
- moved C4 33.0 mm to (155.1, 101.1)
- moved C2 29.2 mm to (149.5, 101.1)
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Connections:
- D3 pad 2: +5V -> Net-(D3-A)
- J4 pad A4: +5V -> Net-(D3-A)
- J4 pad A9: +5V -> Net-(D3-A)
- J4 pad B4: +5V -> Net-(D3-A)
- J4 pad B9: +5V -> Net-(D3-A)
Routing:
- net +3V3: track 0.00 -> 398.6 mm, vias 0 -> 4
- net STS_SIG: track 0.00 -> 213.8 mm, vias 0 -> 3
- net +5V: track 31.4 -> 242.0 mm, vias 0 -> 4
- net I2C1_SCL: track 0.00 -> 210.2 mm, vias 0 -> 2
- net I2C1_SDA: track 0.00 -> 201.0 mm, vias 0 -> 3
- net GND: track 21.1 -> 186.1 mm, vias 0 -> 46
- net Net-(D8-A): track 25.9 -> 178.9 mm, vias 0 -> 1
- net XSHUT1: track 0.00 -> 85.1 mm, vias 0 -> 2
- net Net-(D7-A): track 20.8 -> 103.7 mm, vias 0 -> 1
- net XSHUT2: track 0.00 -> 82.2 mm, vias 0 -> 1
- net UART2_TX: track 0.00 -> 78.3 mm, vias 0 -> 2
- net UART2_RX: track 0.00 -> 75.9 mm, vias 0 -> 2
- net UART4_RX: track 0.00 -> 69.8 mm, vias 0 -> 1
- net UART4_TX: track 0.00 -> 68.8 mm, vias 0 -> 1
- net VDD: track 4.68 -> 68.7 mm
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- added copper zone on B.Cu, net GND
- added copper zone on F.Cu, net GND
Other:
- board size 130 x 136 mm -> 130 x 146 mm

Commit message: つかれた
Parts:
- added G***: LOGO, logo:st_logo_big, F.Cu at (160.7, 100.9)
- added G***: LOGO, logo:tuton_logo_big, F.Cu at (126.5, 100.3)
- added G***: LOGO, logo:jlcpcb_logo_big, F.Cu at (146.0, 99.7)
Other:
- board text added: "+"
- board text added: "1"
- board text added: "220uF"
- board text added: "3V3"
- board text added: "5V"
- board text added: "BACK"
- board text added: "BNO055"
- board text added: "BOOT"
- board text added: "CH340E"
- board text added: "FRONT"
- board text added: "G"
- board text added: "GND"
- board text added: "LINE"
- board text added: "MAX485"
- board text added: "RST"
- board text added: "RX"
- board text added: "S"
- board text added: "STM32F446RE"
- board text added: "TOP"
- board text added: "TX"
- board text added: "Tuton 2025 NAGOYA 01-MAIN"
- board text added: "V"
- board text added: "VDD"
- board text added: "X"
- board text added: "XSHUT1"
- board text added: "XSHUT2"
