File: 1-TOKYO/08-REG_mod/08-REG_mod.kicad_pcb (KiCad board)
At the start: 2 copper layers, 19.7 x 26.7 mm, 13 parts, among them J1 Conn_01x05, U1 TPS5430DDA

Commit message: readme
Parts:
- J1: footprint Connector_PinHeader_2.54mm:PinHeader_1x05_P2.54mm_Horizontal -> Connector_PinHeader_2.54mm:PinHeader_1x05_P2.54mm_Vertical; moved to B.Cu
- turned J1 to 90 degrees
